File: esp32-e22/esp32-e22.kicad_pcb (KiCad board)
At the start: 2 copper layers, 71.1 x 102.9 mm, 31 parts, among them J1 Conn_01x04_Socket, J10 Conn_01x02_Socket, J3 Conn_01x04_Socket, J4 Conn_01x03_Socket, J5 SMA, J6 Conn_01x02_Socket, J7 USB_C_Receptacle_PowerOnly_6P, J8 Conn_01x04_Socket, J9 Conn_01x02_Socket, SW1 SW_Push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

Commit message: update footprint of sma connector
Parts:
- J5: footprint Connector_Coaxial:SMA_Amphenol_901-143_Horizontal -> Connector_Coaxial:SMA_Amphenol_901-144_Vertical
- moved D1 32.1 mm to (198.2, 49.0)
- moved D2 32.1 mm to (198.8, 54.1)
Changed lines of the file:
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@@
 	(footprint "Diode_THT:D_A-405_P7.62mm_Horizontal"
 		(layer "F.Cu")
-		(at 187.96 79.375)
+		(at 198.19 49)
 		(descr "Diode, A-405 series, Axial, Horizontal, pin pitch=7.62mm, , length*diameter=5.2*2.7mm^2, , http://www.diodes.com/_files/packages/A-405.pdf")
 		(tags "Diode A-405 series Axial Horizontal pin pitch 7.62mm  length 5.2mm diameter 2.7mm")
@@
 		)
 	)
-	(footprint "Connector_Coaxial:SMA_Amphenol_901-143_Horizontal"
+	(footprint "Connector_Coaxial:SMA_Amphenol_901-144_Vertical"
 		(layer "F.Cu")
 		(at 124.46 48.54)
-		(descr " Amphenol RF 901-143 https://www.amphenolrf.com/library/download/link/link_id/585682")
-		(tags "SMA THT Female Jack Horizontal")
+		(descr "https://www.amphenolrf.com/downloads/dl/file/id/7023/product/3103/901_144_customer_drawing.pdf")
+		(tags "SMA THT Female Jack Vertical")
 		(property "Reference" "J5"
-			(at -5.2 0 90)
+			(at 0 -4.75 0)
 			(layer "F.SilkS")
 			(effects
@@
 			)
 		)
-		(property "Footprint" "Connector_Coaxial:SMA_Amphenol_901-143_Horizontal"
+		(property "Footprint" "Connector_Coaxial:SMA_Amphenol_901-144_Vertical"
 			(at 0 0 0)
 			(unlocked yes)
@@
 		(attr through_hole)
 		(fp_line
-			(start -4.1 -4.1)
-			(end -4.1 4.1)
+			(start -3.355 -1.45)
+			(end -3.355 1.45)
 			(stroke
 				(width 0.12)
@@
 		)
 		(fp_line
-			(start -4.1 -4.1)
-			(end 4.1 -4.1)
+			(start -1.45 -3.355)
+			(end 1.45 -3.355)
 			(stroke
 				(width 0.12)
@@
 		)
 		(fp_line
-			(start -4.1 0.5)
-			(end -3.6 0)
+			(start -1.45 3.355)
+			(end 1.45 3.355)
 			(stroke
 				(width 0.12)
@@
 		)
 		(fp_line
-			(start -4.1 4.1)
-			(end 4.1 4.1)
+			(start 3.355 -1.45)
+			(end 3.355 1.45)
 			(stroke
 				(width 0.12)
@@
 		)
 		(fp_line
-			(start -3.6 0)
-			(end -4.1 -0.5)
-			(stroke
-				(width 0.12)
-				(type solid)
-			)
-			(layer "F.SilkS")
-		)
-		(fp_line
-			(start 4.1 -4.1)
-			(end 4.1 4.1)
-			(stroke
-				(width 0.12)
-				(type solid)
-			)
-			(layer "F.SilkS")
-		)
-		(fp_line
-			(start -4.3 -12)
-			(end -4.3 4.3)
+			(start -4.17 -4.17)
+			(end -4.17 4.17)
 			(stroke
 				(width 0.05)
@@
 		)
 		(fp_line
-			(start -4.3 -12)
-			(end 4.3 -12)
+			(start -4.17 -4.17)
+			(end 4.17 -4.17)
 			(stroke
 				(width 0.05)
@@
 		)
 		(fp_line
-			(start 4.3 4.3)
-			(end -4.3 4.3)
+			(start 4.17 4.17)
+			(end -4.17 4.17)
 			(stroke
 				(width 0.05)
@@
 		)
 		(fp_line
-			(start 4.3 4.3)
-			(end 4.3 -12)
+			(start 4.17 4.17)
+			(end 4.17 -4.17)
 			(stroke
 				(width 0.05)
@@
 		)
 		(fp_line
-			(start -3.5 -3.5)
-			(end -3.5 3.5)
-			(stroke
-				(width 0.1)
-				(type solid)
-			)
-			(layer "F.Fab")
-		)
-		(fp_line
-			(start -3.5 -3.5)
-			(end 3.5 -3.5)
-			(stroke
-				(width 0.1)
-				(type solid)
-			)
-			(layer "F.Fab")
-		)
-		(fp_line
-			(start -3.5 -1)
-			(end -2.5 0)
-			(stroke
-				(width 0.1)
-				(type solid)
-			)
-			(layer "F.Fab")
-		)
-		(fp_line
-			(start -3.5 3.5)
-			(end 3.5 3.5)
+			(start -3.175 -3.175)
+			(end -3.175 3.175)
 			(stroke
 				(width 0.1)
@@
 		)
 		(fp_line
-			(start -3 -9.5)
-			(end 3 -10)
+			(start -3.175 -3.175)
+			(end 3.175 -3.175)
 			(stroke
 				(width 0.1)
@@
 		)
 		(fp_line
-			(start -3 -9)
-			(end 3 -9.5)
+			(start -3.175 3.175)
+			(end 3.175 3.175)
 			(stroke
 				(width 0.1)
@@
 		)
 		(fp_line
-			(start -3 -8.5)
-			(end 3 -9)
+			(start 3.175 -3.175)
+			(end 3.175 3.175)
 			(stroke
 				(width 0.1)
@@
 			(layer "F.Fab")
 		)
-		(fp_line
-			(start -3 -8)
-			(end 3 -8.5)
-			(stroke
-				(width 0.1)
-				(type solid)
-			)
-			(layer "F.Fab")
-		)
-		(fp_line
-			(start -3 -7.5)
-			(end 3 -8)
-			(stroke
-				(width 0.1)
-				(type solid)
-			)
-			(layer "F.Fab")
-		)
-		(fp_line
-			(start -3 -7)
-			(end 3 -7.5)
-			(stroke
-				(width 0.1)
-				(type solid)
-			)
-			(layer "F.Fab")
-		)
-		(fp_line
-			(start -3 -5.5)
-			(end -3 -3.5)
-			(stroke
-				(width 0.1)
-				(type solid)
-			)
-			(layer "F.Fab")
-		)
-		(fp_line
-			(start -2.5 -11.5)
-			(end -2.5 -5.5)
-			(stroke
-				(width 0.1)
-				(type solid)
-			)
-			(layer "F.Fab")
-		)
-		(fp_line
-			(start -2.5 -11.5)
-			(end 2.5 -11.5)
-			(stroke
-				(width 0.1)
-				(type solid)
-			)
-			(layer "F.Fab")
-		)
-		(fp_line
-			(start -2.5 0)
-			(end -3.5 1)
-			(stroke
-				(width 0.1)
-				(type solid)
-			)
-			(layer "F.Fab")
-		)
-		(fp_line
-			(start 2.5 -11.5)
-			(end 2.5 -5.5)
-			(stroke
-				(width 0.1)
-				(type solid)
-			)
-			(layer "F.Fab")
-		)
-		(fp_line
-			(start 3 -5.5)
-			(end -3 -5.5)
-			(stroke
-				(width 0.1)
-				(type solid)
-			)
-			(layer "F.Fab")
-		)
-		(fp_line
-			(start 3 -5.5)
-			(end 3 -3.5)
-			(stroke
-				(width 0.1)
-				(type solid)
-			)
-			(layer "F.Fab")
-		)
-		(fp_line
-			(start 3.5 -3.5)
-			(end 3.5 3.5)
+		(fp_circle
+			(center 0 0)
+			(end 3.175 0)
 			(stroke
 				(width 0.1)
 				(type solid)
 			)
+			(fill none)
 			(layer "F.Fab")
 		)
@@
 			)
 		)
-		(pad "1" thru_hole roundrect
+		(pad "1" thru_hole circle
 			(at 0 0)
-			(size 2.3 2.3)
+			(size 2.05 2.05)
 			(drill 1.5)
 			(layers "*.Cu" "*.Mask")
-			(remove_unused_layers yes)
-			(keep_end_layers yes)
-			(zone_layer_connections)
-			(roundrect_rratio 0.087)
+			(remove_unused_layers no)
 			(net 10 "Net-(J5-In)")
 			(pinfunction "In")
@@
 		(pad "2" thru_hole circle
 			(at -2.54 -2.54)
-			(size 2.5 2.5)
+			(size 2.25 2.25)
 			(drill 1.7)
 			(layers "*.Cu" "*.Mask")
-			(remove_unused_layers yes)
-			(keep_end_layers yes)
-			(zone_layer_connections)
+			(remove_unused_layers no)
 			(net 3 "GND")
 			(pinfunction "Ext")
@@
 		(pad "2" thru_hole circle
 			(at -2.54 2.54)
-			(size 2.5 2.5)
+			(size 2.25 2.25)
 			(drill 1.7)
 			(layers "*.Cu" "*.Mask")
-			(remove_unused_layers yes)
-			(keep_end_layers yes)
-			(zone_layer_connections)
+			(remove_unused_layers no)
 			(net 3 "GND")
 			(pinfunction "Ext")
@@
 		(pad "2" thru_hole circle
 			(at 2.54 -2.54)
-			(size 2.5 2.5)
+			(size 2.25 2.25)
 			(drill 1.7)
 			(layers "*.Cu" "*.Mask")
-			(remove_unused_layers yes)
-			(keep_end_layers yes)
-			(zone_layer_connections)
+			(remove_unused_layers no)
 			(net 3 "GND")
 			(pinfunction "Ext")
@@
 		(pad "2" thru_hole circle
 			(at 2.54 2.54)
-			(size 2.5 2.5)
+			(size 2.25 2.25)
 			(drill 1.7)
 			(layers "*.Cu" "*.Mask")
-			(remove_unused_layers yes)
-			(keep_end_layers yes)
-			(zone_layer_connections)
+			(remove_unused_layers no)
 			(net 3 "GND")
 			(pinfunction "Ext")
@@
 	(footprint "Diode_SMD:D_SOD-523"
 		(layer "F.Cu")
-		(at 188.595 84.455)
+		(at 198.825 54.08)
 		(descr "http://www.diodes.com/datasheets/ap02001.pdf p.144")
 		(tags "Diode SOD523")

Commit message: update to v2.0.9
Parts:
- added D3: 1N5817, Diode_THT:D_DO-41_SOD81_P7.62mm_Horizontal, F.Cu at (154.9, 125.7)
- added REF**: MountingHole_2.2mm_M2_Pad_TopBottom, MountingHole:MountingHole_2.2mm_M2_Pad_TopBottom, F.Cu at (175.3, 63.5)
- added REF**: MountingHole_2.2mm_M2_Pad_TopBottom, MountingHole:MountingHole_2.2mm_M2_Pad_TopBottom, F.Cu at (115.6, 138.4)
- added REF**: MountingHole_2.2mm_M2_Pad_TopBottom, MountingHole:MountingHole_2.2mm_M2_Pad_TopBottom, F.Cu at (115.6, 63.5)
- added REF**: MountingHole_2.2mm_M2_Pad_TopBottom, MountingHole:MountingHole_2.2mm_M2_Pad_TopBottom, F.Cu at (175.3, 138.4)
- C1, C7: footprint Capacitor_THT:CP_Radial_D8.0mm_P5.00mm -> Capacitor_THT:CP_Radial_D5.0mm_P2.50mm
- D1: value D_Schottky_Small -> 1N5817; footprint Diode_THT:D_A-405_P7.62mm_Horizontal -> Diode_THT:D_DO-41_SOD81_P7.62mm_Horizontal
- D2: value SD05_SOD323 -> LESD5D5.0CT1G
- J5: footprint Connector_Coaxial:SMA_Amphenol_901-144_Vertical -> Connector_Coaxial:SMA_Amphenol_132134-14_Vertical
- JP1, JP2, R6, R7: moved to B.Cu
- moved D1 78.3 mm to (163.8, 119.4)
- moved D2 76.3 mm to (159.3, 119.4)
- moved R6 42.1 mm to (162.6, 106.7)
- moved R7 42.1 mm to (162.6, 102.9)
- moved J6 20.3 mm to (157.5, 86.4), turned to 0 degrees
- moved C7 14.6 mm to (154.3, 121.9), turned to 90 degrees
- moved J5 13.2 mm to (137.2, 52.1)
- moved C1 12.8 mm to (162.6, 87.6)
- moved U1 12.7 mm to (145.1, 70.6)
- moved JP2 12.7 mm to (165.1, 99.1), turned to 90 degrees
- moved C2 11.5 mm to (170.2, 87.6)
- moved JP1 7.62 mm to (162.6, 96.5), turned to -90 degrees
- moved C4 6.51 mm to (170.2, 74.9)
- moved J9 5.24 mm to (171.4, 127.0)
- moved J8 4.03 mm to (170.2, 71.1)
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Connections:
- D1 pad 1: unconnected-(D1-K-Pad1) -> +5V
- D1 pad 2: unconnected-(D1-A-Pad2) -> Net-(D1-A)
- D2 pad 1: unconnected-(D2-A1-Pad1) -> GND
- D2 pad 2: unconnected-(D2-A2-Pad2) -> +5V
- J7 pad A9: +5V -> Net-(D3-A)
- J7 pad B9: +5V -> Net-(D3-A)
- J9 pad 1: +5V -> Net-(D1-A)
Routing:
- net +5V: track 149.3 -> 113.6 mm
- net Net-(D3-A): track 0.00 -> 14.1 mm
- net Net-(J6-Pin_1): track 12.6 -> 3.91 mm
- net /GPS_RX: track 36.3 -> 44.2 mm
- net Net-(D1-A): track 0.00 -> 7.62 mm
- net +3.3V: track 128.4 -> 135.9 mm, vias 0 -> 1
- net /E22_BUSY: track 75.6 -> 82.1 mm
- net /E22_NRST: track 76.0 -> 82.1 mm
- net /E22_DIO1: track 74.1 -> 79.5 mm
- net /E22_TXEN: track 61.1 -> 66.4 mm
- net /E22_NSS: track 71.3 -> 66.2 mm
- net /E22_SCK: track 67.7 -> 62.6 mm
- net Net-(U2-CHIP_PU): track 18.9 -> 13.8 mm
- net /GPS_TX: track 36.3 -> 40.6 mm
- net /E22_RXEN: track 53.5 -> 57.8 mm
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Other:
- board size 71.1 x 102.9 mm -> 69.9 x 97.8 mm
