File: esp32-e22/esp32-e22.kicad_sch (KiCad schematic)
At the start: 29 parts, among them J1 Conn_01x04_Socket, J10 Conn_01x02_Socket, J3 Conn_01x04_Socket, J4 Conn_01x03_Socket, J5 SMA, J6 Conn_01x02_Socket, J7 USB_C_Receptacle_PowerOnly_6P, J8 Conn_01x04_Socket, J9 Conn_01x02_Socket, SW1 SW_Push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

Commit message: update to v2.0.8
Parts:
- added D1: D_Schottky_Small, Diode_THT:D_A-405_P7.62mm_Horizontal, symbol Device:D_Schottky_Small
- added D2: SD05_SOD323, Diode_SMD:D_SOD-523, symbol Diode:SD05_SOD323
Changed lines of the file:
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@@
 		(title "ESP32 - E22 Board")
 		(date "2024-10-04")
-		(rev "V2.0.7")
+		(rev "V2.0.8")
 		(company "DK9BT / OE3WAS")
 	)
@@
 	)
 	(symbol
+		(lib_id "Device:D_Schottky_Small")
+		(at 132.08 172.72 0)
+		(unit 1)
+		(exclude_from_sim no)
+		(in_bom yes)
+		(on_board yes)
+		(dnp no)
+		(fields_autoplaced yes)
+		(property "Reference" "D1"
+			(at 131.826 166.37 0)
+			(effects
+				(font
+					(size 1.27 1.27)
+				)
+			)
+		)
+		(property "Value" "D_Schottky_Small"
+			(at 131.826 168.91 0)
+			(effects
+				(font
+					(size 1.27 1.27)
+				)
+			)
+		)
+		(property "Footprint" "Diode_THT:D_A-405_P7.62mm_Horizontal"
+			(at 132.08 172.72 90)
+			(effects
+				(font
+					(size 1.27 1.27)
+				)
+				(hide yes)
+			)
+		)
+		(property "Datasheet" "~"
+			(at 132.08 172.72 90)
+			(effects
+				(font
+					(size 1.27 1.27)
+				)
+				(hide yes)
+			)
+		)
+		(property "Description" "Schottky diode, small symbol"
+			(at 132.08 172.72 0)
+			(effects
+				(font
+					(size 1.27 1.27)
+				)
+				(hide yes)
+			)
+		)
+		(pin "2"
+		)
+		(pin "1"
+		)
+		(instances
+			(project ""
+				(path "/7ac59502-473d-4014-a9ef-f4cf3cefb926"
+					(reference "D1")
+					(unit 1)
+				)
+			)
+		)
+	)
+	(symbol
 		(lib_id "Connector:Conn_01x04_Socket")
 		(at 190.5 93.98 0)
@@
 					(unit 1)
 				)
+			)
+		)
+	)
+	(symbol
+		(lib_id "Diode:SD05_SOD323")
+		(at 95.25 181.61 0)
+		(unit 1)
+		(exclude_from_sim no)
+		(in_bom yes)
+		(on_board yes)
+		(dnp no)
+		(fields_autoplaced yes)
+		(property "Reference" "D2"
+			(at 95.25 175.26 0)
+			(effects
+				(font
+					(size 1.27 1.27)
+				)
+			)
+		)
+		(property "Value" "SD05_SOD323"
+			(at 95.25 177.8 0)
+			(effects
+				(font
+					(size 1.27 1.27)
+				)
+			)
+		)
+		(property "Footprint" "Diode_SMD:D_SOD-523"
+			(at 95.25 186.69 0)
+			(effects
+				(font
+					(size 1.27 1.27)
+				)
+				(hide yes)
+			)
+		)
+		(property "Datasheet" "https://www.littelfuse.com/~/media/electronics/datasheets/tvs_diode_arrays/littelfuse_tvs_diode_array_sd_c_datasheet.pdf.pdf"
+			(at 95.25 181.61 0)
+			(effects
+				(font
+					(size 1.27 1.27)
+				)
+				(hide yes)
+			)
+		)
+		(property "Description" "5V, 450W Discrete Bidirectional TVS Diode, SOD-323"
+			(at 95.25 181.61 0)
+			(effects
+				(font
+					(size 1.27 1.27)
+				)
+				(hide yes)
+			)
+		)
+		(pin "1"
+		)
+		(pin "2"
+		)
+		(instances
+			(project ""
+				(path "/7ac59502-473d-4014-a9ef-f4cf3cefb926"
+					(reference "D2")
+					(unit 1)
+				)

Commit message: update to v2.0.9
Parts:
- added D3: 1N5817, Diode_THT:D_DO-41_SOD81_P7.62mm_Horizontal, symbol Device:D_Schottky_Small
- C1, C7: footprint Capacitor_THT:CP_Radial_D8.0mm_P5.00mm -> Capacitor_THT:CP_Radial_D5.0mm_P2.50mm
- D1: value D_Schottky_Small -> 1N5817; footprint Diode_THT:D_A-405_P7.62mm_Horizontal -> Diode_THT:D_DO-41_SOD81_P7.62mm_Horizontal
- D2: value SD05_SOD323 -> LESD5D5.0CT1G
- J5: footprint Connector_Coaxial:SMA_Amphenol_901-143_Horizontal -> Connector_Coaxial:SMA_Amphenol_132134-14_Vertical
Connections:
- net +5V: now also D1.1 (K), D2.2 (A2), D3.1 (K); no longer J7.A9 (VBUS), J7.B9 (VBUS), J9.1 (Pin_1)
- net GND: now also D2.1 (A1)
- net at D1.2 (A): now also J9.1 (Pin_1)
- new net: D3.2 (A), J7.A9 (VBUS), J7.B9 (VBUS)
Other:
- moved on the sheet: C1, C2, C3, C7, D1, D2, J7, J9, R1, R2
