File: ESP32-E22_V2.1/KiCad/esp32-e22.kicad_pcb (KiCad board)
At the start: 2 copper layers, 70 x 99 mm, 38 parts, among them J1 Conn_01x02_Socket, J3 Conn_01x02_Socket, J4 Conn_01x04_Socket, J5 Conn_01x03_Socket, J6 Conn_01x04_Socket, J7 Conn_01x04_Socket, J8 SMA, J9 Conn_01x02_Socket, SW1 SW_Push, U1 ESP32-DevKitC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

Commit message: some fixes
Parts:
- added NT1: NetTie_2, NetTie:NetTie-2_SMD_Pad0.5mm, B.Cu at (165.9, 94.6)
Connections:
- JP1 pad 1: Net-(JP1-A) -> +3.3V
- JP2 pad 2: GND -> Net-(JP2-A)
- U2 pad 1: Net-(JP1-A) -> +3.3V
Routing:
- net +3.3V: track 159.5 -> 165.9 mm
- net Net-(JP2-A): track 7.47 -> 12.0 mm
- net Net-(JP1-A): track 3.88 -> 0.00 mm
Changed lines of the file:
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@@
 	(net 39 "/E22_TXEN")
 	(net 40 "unconnected-(U1-U0TXD{slash}GPIO1-Pad35)")
-	(net 41 "Net-(JP1-A)")
-	(net 42 "Net-(JP2-A)")
-	(net 43 "Net-(D1-A)")
-	(net 44 "Net-(U3-ANT)")
-	(net 45 "Net-(J2-CC2)")
-	(net 46 "Net-(J2-CC1)")
+	(net 41 "Net-(JP2-A)")
+	(net 42 "Net-(D1-A)")
+	(net 43 "Net-(U3-ANT)")
+	(net 44 "Net-(J2-CC2)")
+	(net 45 "Net-(J2-CC1)")
 	(footprint "Connector_PinHeader_2.54mm:PinHeader_1x03_P2.54mm_Vertical"
 		(layer "F.Cu")
@@
 			(layers "*.Cu" "*.Mask")
 			(remove_unused_layers no)
-			(net 46 "Net-(J2-CC1)")
+			(net 45 "Net-(J2-CC1)")
 			(pintype "passive")
 		)
@@
 			(layer "F.Fab")
 		)
+		(pad "" np_thru_hole circle
+			(at -11 -11)
+			(size 3 3)
+			(drill 2)
+			(layers "F&B.Cu" "*.Mask")
+			(solder_mask_margin 0.102)
+		)
+		(pad "" np_thru_hole circle
+			(at -11 11)
+			(size 3 3)
+			(drill 2)
+			(layers "F&B.Cu" "*.Mask")
+			(solder_mask_margin 0.102)
+		)
+		(pad "" np_thru_hole circle
+			(at 11 -11)
+			(size 3 3)
+			(drill 2)
+			(layers "F&B.Cu" "*.Mask")
+			(solder_mask_margin 0.102)
+		)
+		(pad "" np_thru_hole circle
+			(at 11 11)
+			(size 3 3)
+			(drill 2)
+			(layers "F&B.Cu" "*.Mask")
+			(solder_mask_margin 0.102)
+		)
 		(pad "1" thru_hole rect
 			(at -3.81 -11.5)
@@
 			(layers "*.Cu" "*.Mask")
 			(remove_unused_layers no)
-			(net 41 "Net-(JP1-A)")
+			(net 2 "+3.3V")
 			(pinfunction "VCC_IN")
 			(pintype "input")
@@
 			(layers "*.Cu" "*.Mask")
 			(remove_unused_layers no)
-			(net 42 "Net-(JP2-A)")
+			(net 41 "Net-(JP2-A)")
 			(pinfunction "GND")
 			(pintype "input")
@@
 			(solder_mask_margin 0.102)
 		)
-		(pad "S1" thru_hole circle
-			(at -11 -11)
-			(size 3 3)
-			(drill 2)
-			(layers "*.Cu" "*.Mask")
-			(remove_unused_layers no)
-			(solder_mask_margin 0.102)
-		)
-		(pad "S2" thru_hole circle
-			(at 11 -11)
-			(size 3 3)
-			(drill 2)
-			(layers "*.Cu" "*.Mask")
-			(remove_unused_layers no)
-			(solder_mask_margin 0.102)
-		)
-		(pad "S3" thru_hole circle
-			(at 11 11)
-			(size 3 3)
-			(drill 2)
-			(layers "*.Cu" "*.Mask")
-			(remove_unused_layers no)
-			(solder_mask_margin 0.102)
-		)
-		(pad "S4" thru_hole circle
-			(at -11 11)
-			(size 3 3)
-			(drill 2)
-			(layers "*.Cu" "*.Mask")
-			(remove_unused_layers no)
-			(solder_mask_margin 0.102)
-		)
 		(model "${KIPRJMOD}/3D_model/DM-OLED096-636.step"
 			(offset
@@
 			(layers "*.Cu" "*.Mask")
 			(remove_unused_layers no)
-			(net 43 "Net-(D1-A)")
+			(net 42 "Net-(D1-A)")
 			(pinfunction "V+")
 			(pintype "output")
@@
 			(layers "*.Cu" "*.Mask")
 			(remove_unused_layers no)
-			(net 46 "Net-(J2-CC1)")
+			(net 45 "Net-(J2-CC1)")
 			(pinfunction "CC1")
 			(pintype "passive")
@@
 			(layers "*.Cu" "*.Mask")
 			(remove_unused_layers no)
-			(net 45 "Net-(J2-CC2)")
+			(net 44 "Net-(J2-CC2)")
 			(pinfunction "CC2")
 			(pintype "passive")
@@
 			(layers "*.Cu" "*.Mask")
 			(remove_unused_layers no)
-			(net 43 "Net-(D1-A)")
+			(net 42 "Net-(D1-A)")
 			(pinfunction "A")
 			(pintype "passive")
@@
 			(layers "F.Cu" "F.Paste" "F.Mask")
 			(roundrect_rratio 0.1666666667)
-			(net 44 "Net-(U3-ANT)")
+			(net 43 "Net-(U3-ANT)")
 			(pinfunction "ANT")
 			(pintype "bidirectional")
@@
 			(layers "*.Cu" "*.Mask")
 			(remove_unused_layers no)
-			(net 45 "Net-(J2-CC2)")
+			(net 44 "Net-(J2-CC2)")
 			(pintype "passive")
 		)
@@
 			(layers "*.Cu" "*.Mask")
 			(remove_unused_layers no)
-			(net 41 "Net-(JP1-A)")
+			(net 2 "+3.3V")
 			(pinfunction "A")
 			(pintype "passive")
@@
 			(layers "B.Cu" "B.Paste" "B.Mask")
 			(roundrect_rratio 0.243902)
-			(net 44 "Net-(U3-ANT)")
+			(net 43 "Net-(U3-ANT)")
 			(pintype "passive")
 		)
@@
 			(layers "*.Cu" "*.Mask")
 			(remove_unused_layers no)
-			(net 42 "Net-(JP2-A)")
+			(net 41 "Net-(JP2-A)")
 			(pinfunction "A")
 			(pintype "passive")
@@
 			(layers "*.Cu" "*.Mask")
 			(remove_unused_layers no)
-			(net 3 "GND")
+			(net 41 "Net-(JP2-A)")
 			(pinfunction "B")
 			(pintype "passive")
 		)
 	)
+	(footprint "NetTie:NetTie-2_SMD_Pad0.5mm"
+		(layer "B.Cu")
+		(at 165.87 94.63)
+		(descr "Net tie, 2 pin, 0.5mm square SMD pads")
+		(tags "net tie")
+		(property "Reference" "NT1"
+			(at 0 1.2 360)
+			(layer "B.SilkS")
+			(hide yes)
+			(effects
+				(font
+					(size 1 1)
+					(thickness 0.15)
+				)
+				(justify mirror)
+			)
+		)
+		(property "Value" "NetTie_2"
+			(at 0 -1.2 360)
+			(layer "B.Fab")
+			(hide yes)
+			(effects
+				(font
+					(size 1 1)
+					(thickness 0.15)
+				)
+				(justify mirror)
+			)
+		)
+		(property "Footprint" "NetTie:NetTie-2_SMD_Pad0.5mm"
+			(at 0 0 180)
+			(unlocked yes)
+			(layer "B.Fab")
+			(hide yes)
+			(effects
+				(font
+					(size 1.27 1.27)
+					(thickness 0.15)
+				)
+				(justify mirror)
+			)
+		)
+		(property "Datasheet" ""
+			(at 0 0 180)
+			(unlocked yes)
+			(layer "B.Fab")
+			(hide yes)
+			(effects
+				(font
+					(size 1.27 1.27)
+					(thickness 0.15)
+				)
+				(justify mirror)
+			)
+		)
+		(property "Description" "Net tie, 2 pins"
+			(at 0 0 180)
+			(unlocked yes)
+			(layer "B.Fab")
+			(hide yes)
+			(effects
+				(font
+					(size 1.27 1.27)
+					(thickness 0.15)
+				)
+				(justify mirror)
+			)
+		)
+		(property ki_fp_filters "Net*Tie*")
+		(sheetname "Stammblatt")
+		(sheetfile "esp32-e22.kicad_sch")
+		(attr exclude_from_pos_files exclude_from_bom allow_missing_courtyard)
+		(net_tie_pad_groups "1, 2")
+		(fp_poly
+			(pts
+				(xy -0.5 0.25) (xy 0.5 0.25) (xy 0.5 -0.25) (xy -0.5 -0.25)
+			)
+			(stroke
+				(width 0)
+				(type solid)
+			)
+			(fill solid)
+			(layer "B.Cu")
+		)
+		(pad "1" smd circle
+			(at -0.5 0)
+			(size 0.5 0.5)
+			(layers "B.Cu")
+			(net 41 "Net-(JP2-A)")
+			(pinfunction "1")
+			(pintype "passive")
+		)
+		(pad "2" smd circle
+			(at 0.5 0)
+			(size 0.5 0.5)
+			(layers "B.Cu")
+			(net 3 "GND")
+			(pinfunction "2")
+			(pintype "passive")
+		)
+	)
 	(footprint "Resistor_THT:R_Axial_DIN0207_L6.3mm_D2.5mm_P7.62mm_Horizontal"
 		(layer "B.Cu")
@@
 	)
 	(segment
+		(start 162.56 96.52)
+		(end 162.56 92.64)
+		(width 0.3)
+		(layer "B.Cu")
+		(net 2)
+	)
+	(segment
 		(start 170.22 78.71)
 		(end 170.19 78.74)
@@
 	)
 	(segment
+		(start 162.56 96.52)
+		(end 162.56 99.06)
+		(width 0.2)
+		(layer "B.Cu")
+		(net 2)
+	)
+	(segment
 		(start 170.19 74.9)
 		(end 170.22 74.93)
@@
 	)
 	(segment
-		(start 162.56 96.52)
-		(end 162.56 92.64)
-		(width 0.3)
+		(start 165.1 96.52)
+		(end 165.1 99.06)
+		(width 0.2)
+		(layer "B.Cu")
+		(net 41)
+	)
+	(segment
+		(start 165.1 94.9)
+		(end 165.37 94.63)
+		(width 0.2)
 		(layer "B.Cu")
 		(net 41)
@@
 		(width 0.3)
 		(layer "B.Cu")
-		(net 42)
+		(net 41)
+	)
+	(segment
+		(start 165.1 96.52)
+		(end 165.1 94.9)
+		(width 0.2)
+		(layer "B.Cu")
+		(net 41)
 	)
 	(segment
@@
 		(width 0.3)
 		(layer "B.Cu")
-		(net 42)
+		(net 41)
 	)
 	(segment
@@
 		(width 0.3)
 		(layer "B.Cu")
-		(net 42)
+		(net 41)
 	)
 	(segment
@@
 		(width 1)
 		(layer "F.Cu")
-		(net 43)
+		(net 42)
 	)
 	(segment
@@
 		(width 1)
 		(layer "F.Cu")
-		(net 43)
+		(net 42)
 	)
 	(segment
@@
 		(width 1)
 		(layer "F.Cu")
-		(net 43)
+		(net 42)
 	)
 	(segment
@@
 		(width 0.3)
 		(layer "F.Cu")
-		(net 44)
+		(net 43)
 	)
 	(segment
@@
 		(width 0.3)
 		(layer "F.Cu")
-		(net 44)
+		(net 43)
 	)
 	(segment
@@
 		(width 0.3)
 		(layer "F.Cu")
-		(net 44)
+		(net 43)
 	)
 	(via
@@
 		(drill 0.3)
 		(layers "F.Cu" "B.Cu")
-		(net 44)
+		(net 43)
 	)
 	(segment
@@
 		(width 1)
 		(layer "B.Cu")
-		(net 44)
+		(net 43)
 	)
 	(segment
@@
 		(width 0.3)
 		(layer "B.Cu")
-		(net 45)
+		(net 44)
 	)
 	(segment
@@
 		(width 0.3)
 		(layer "B.Cu")
-		(net 45)
+		(net 44)
 	)
 	(segment
@@
 		(width 0.3)
 		(layer "B.Cu")
-		(net 46)
+		(net 45)
 	)
 	(segment
@@
 		(width 0.3)
 		(layer "B.Cu")
-		(net 46)
+		(net 45)
 	)
 	(zone

Commit message: update
Parts:
- NT1: moved to F.Cu
- moved NT1 0.81 mm to (165.1, 94.7), turned to 180 degrees
Routing:
- net Net-(JP2-A): track 12.0 -> 15.6 mm
