File: ESP32-E22_V2.1/KiCad/esp32-e22.kicad_pcb (KiCad board)
At the start: 2 copper layers, 70 x 99 mm, 39 parts, among them J1 Conn_01x02_Socket, J3 Conn_01x02_Socket, J4 Conn_01x04_Socket, J5 Conn_01x03_Socket, J6 Conn_01x04_Socket, J7 Conn_01x04_Socket, J8 SMA, J9 Conn_01x02_Socket, SW1 SW_Push, U1 ESP32-DevKitC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

Commit message: Beta V2.1.0
Parts:
- moved NT1 0.75 mm to (164.3, 94.6)
Routing:
- net +5V: track 122.4 -> 129.4 mm
- net /MOSI: track 45.3 -> 42.4 mm
- net Net-(JP2-A): track 15.6 -> 13.7 mm
Changed lines of the file:
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@@
 		(title "ESP32+E22 single sided")
 		(date "2024-10-08")
-		(rev "V 2.0.6")
+		(rev "V 2.1.0")
 		(comment 1 "designed by OE3WAS")
 		(comment 4 "AISLER Project ID: LMKJXZAY")
@@
 		(tags "CP Radial series Radial pin pitch 2.50mm  diameter 5mm Electrolytic Capacitor")
 		(property "Reference" "C6"
-			(at 1.25 -3.75 90)
+			(at 3.81 3.175 180)
 			(layer "F.SilkS")
 			(effects
@@
 		(tags "Resistor Axial_DIN0207 series Axial Horizontal pin pitch 7.62mm 0.25W = 1/4W length 6.3mm diameter 2.5mm")
 		(property "Reference" "R4"
-			(at 3.81 -2.37 0)
+			(at -1.905 0 0)
 			(layer "F.SilkS")
 			(effects
@@
 		(tags "Resistor Axial_DIN0207 series Axial Horizontal pin pitch 7.62mm 0.25W = 1/4W length 6.3mm diameter 2.5mm")
 		(property "Reference" "R2"
-			(at 3.81 -2.37 90)
+			(at 0 2.54 180)
 			(layer "F.SilkS")
 			(effects
@@
 		(tags "CP Radial series Radial pin pitch 2.50mm  diameter 6.3mm Electrolytic Capacitor")
 		(property "Reference" "C2"
-			(at 1.25 -4.4 0)
+			(at 6.35 0 0)
 			(layer "F.SilkS")
 			(effects
@@
 		(tags "Through hole pin header THT 1x04 2.54mm single row")
 		(property "Reference" "J7"
-			(at 0 -2.33 90)
+			(at -2.54 2.53 180)
 			(layer "F.SilkS")
 			(effects
@@
 		(at 166.37 104.14)
 		(property "Reference" "U2"
-			(at -9.525 -13.97 0)
+			(at 7.62 -7.62 0)
 			(layer "F.SilkS")
 			(effects
@@
 		(tags "Resistor Axial_DIN0207 series Axial Horizontal pin pitch 7.62mm 0.25W = 1/4W length 6.3mm diameter 2.5mm")
 		(property "Reference" "R5"
-			(at 3.81 -2.37 90)
+			(at 0 -2.37 180)
 			(layer "F.SilkS")
 			(effects
@@
 		(tags "Diode DO-41_SOD81 series Axial Horizontal pin pitch 7.62mm  length 5.2mm diameter 2.7mm")
 		(property "Reference" "D1"
-			(at 3.81 -2.47 90)
+			(at -1.27 -2.54 180)
 			(layer "F.SilkS")
 			(effects
@@
 		(tags "C Disc series Radial pin pitch 5.00mm  diameter 4.7mm width 2.5mm Capacitor")
 		(property "Reference" "C4"
-			(at 2.5 -2.5 90)
+			(at 2.54 2.54 180)
 			(layer "F.SilkS")
 			(effects
@@
 		(tags "THT Terminal Block Phoenix MKDS-1,5-2-5.08 pitch 5.08mm size 10.2x9.8mm^2 drill 1.3mm pad 2.6mm")
 		(property "Reference" "J3"
-			(at 2.54 -6.26 0)
+			(at 0 6.35 0)
 			(layer "F.SilkS")
 			(effects
@@
 		(tags "C Disc series Radial pin pitch 5.00mm  diameter 4.7mm width 2.5mm Capacitor")
 		(property "Reference" "C5"
-			(at 2.5 -2.5 90)
+			(at 7.62 0 180)
 			(layer "F.SilkS")
 			(effects
@@
 		(tags "SMA THT Female Jack Vertical ExtendedLegs")
 		(property "Reference" "J8"
-			(at 0 -4.75 0)
+			(at -5.08 0 0)
 			(layer "F.SilkS")
 			(effects
@@
 		(tags "CP Radial series Radial pin pitch 2.50mm  diameter 5mm Electrolytic Capacitor")
 		(property "Reference" "C3"
-			(at 1.25 -3.75 0)
+			(at 5.08 1.27 0)
 			(layer "F.SilkS")
 			(effects
@@
 	(footprint "NetTie:NetTie-2_SMD_Pad0.5mm"
 		(layer "F.Cu")
-		(at 165.07 94.73 180)
+		(at 164.33 94.615 180)
 		(descr "Net tie, 2 pin, 0.5mm square SMD pads")
 		(tags "net tie")
@@
 		(descr "38.5mm*24mm*3.87mm LoRa Transceiver 33dBm")
 		(property "Reference" "U3"
-			(at 0.02 23.58 90)
+			(at 0.02 23.58 0)
 			(unlocked yes)
 			(layer "F.SilkS")
@@
 		(tags "Through hole pin header THT 1x04 2.54mm single row")
 		(property "Reference" "J4"
-			(at 0 -2.33 90)
+			(at 2.54 2.53 180)
 			(layer "F.SilkS")
 			(effects
@@
 		(tags "C Disc series Radial pin pitch 5.00mm  diameter 4.7mm width 2.5mm Capacitor")
 		(property "Reference" "C1"
-			(at 2.5 -2.5 90)
+			(at -2.54 1.27 180)
 			(layer "F.SilkS")
 			(effects
@@
 		(tags "C Disc series Radial pin pitch 5.00mm  diameter 4.7mm width 2.5mm Capacitor")
 		(property "Reference" "C8"
-			(at 2.5 -2.5 90)
+			(at -2.58 0 180)
 			(layer "F.SilkS")
 			(effects
@@
 		(tags "Resistor Axial_DIN0207 series Axial Horizontal pin pitch 7.62mm 0.25W = 1/4W length 6.3mm diameter 2.5mm")
 		(property "Reference" "R3"
-			(at 3.81 -2.37 0)
+			(at 3.175 -2.37 0)
 			(layer "F.SilkS")
 			(effects
@@
 		(tags "Through hole pin header THT 1x02 2.54mm single row")
 		(property "Reference" "J9"
-			(at 0 -2.33 0)
+			(at -3.81 0 0)
 			(layer "F.SilkS")
 			(effects
@@
 		(tags "Resistor Axial_DIN0207 series Axial Horizontal pin pitch 7.62mm 0.25W = 1/4W length 6.3mm diameter 2.5mm")
 		(property "Reference" "R7"
-			(at 3.81 2.37 0)
+			(at 10.16 0 0)
 			(layer "B.SilkS")
 			(effects
@@
 		(tags "Resistor Axial_DIN0207 series Axial Horizontal pin pitch 7.62mm 0.25W = 1/4W length 6.3mm diameter 2.5mm")
 		(property "Reference" "R6"
-			(at 3.81 2.37 0)
+			(at 10.16 -0.635 0)
 			(layer "B.SilkS")
 			(effects
@@
 	)
 	(segment
-		(start 119.38 76.2)
-		(end 123.19 72.39)
+		(start 167.64 101.6)
+		(end 170.18 104.14)
 		(width 0.3)
 		(layer "F.Cu")
@@
 	)
 	(segment
-		(start 119.38 95.25)
-		(end 119.38 76.2)
+		(start 119.38 76.2)
+		(end 123.19 72.39)
 		(width 0.3)
 		(layer "F.Cu")
@@
 	)
 	(segment
-		(start 167.64 101.6)
-		(end 168.275 101.6)
+		(start 119.38 95.25)
+		(end 119.38 76.2)
 		(width 0.3)
 		(layer "F.Cu")
@@
 	)
 	(segment
-		(start 168.275 101.6)
-		(end 170.18 103.505)
-		(width 0.3)
-		(layer "F.Cu")
-		(net 6)
-	)
-	(segment
 		(start 149.86 101.6)
 		(end 167.64 101.6)
@@
 	)
 	(segment
-		(start 152.4 90.17)
-		(end 147.32 95.25)
+		(start 152.4 97.79)
+		(end 151.13 99.06)
 		(width 0.3)
 		(layer "B.Cu")
@@
 	)
 	(segment
-		(start 147.32 99.06)
-		(end 149.86 99.06)
-		(width 0.3)
-		(layer "B.Cu")
-		(net 14)
-	)
-	(segment
-		(start 147.32 95.25)
-		(end 147.32 99.06)
+		(start 152.4 60.96)
+		(end 152.4 97.79)
 		(width 0.3)
 		(layer "B.Cu")
@@
 	)
 	(segment
-		(start 152.4 60.96)
-		(end 152.4 90.17)
+		(start 151.13 99.06)
+		(end 149.86 99.06)
 		(width 0.3)
 		(layer "B.Cu")
@@
 	)
 	(segment
+		(start 154.94 144.145)
+		(end 144.145 144.145)
+		(width 1)
+		(layer "B.Cu")
+		(net 16)
+	)
+	(segment
 		(start 156.21 135.89)
-		(end 153.67 135.89)
+		(end 156.21 137.16)
 		(width 1)
 		(layer "B.Cu")
@@
 	)
 	(segment
+		(start 156.21 137.16)
+		(end 156.21 142.875)
+		(width 1)
+		(layer "B.Cu")
+		(net 16)
+	)
+	(segment
 		(start 162.56 90.17)
 		(end 162.56 87.63)
@@
 	)
 	(segment
+		(start 144.145 144.145)
+		(end 142.24 142.24)
+		(width 1)
+		(layer "B.Cu")
+		(net 16)
+	)
+	(segment
 		(start 153.67 125.73)
 		(end 154.94 124.46)
@@
 	)
 	(segment
-		(start 160.02 115.57)
-		(end 163.83 119.38)
+		(start 156.21 142.875)
+		(end 154.94 144.145)
 		(width 1)
 		(layer "B.Cu")
@@
 	)
 	(segment
-		(start 153.67 135.89)
-		(end 148.59 135.89)
-		(width 0.5)
+		(start 160.02 115.57)
+		(end 163.83 119.38)
+		(width 1)
 		(layer "B.Cu")
 		(net 16)
@@
 	)
 	(segment
+		(start 156.21 137.16)
+		(end 153.67 137.16)
+		(width 1)
+		(layer "B.Cu")
+		(net 16)
+	)
+	(segment
 		(start 154.94 122.555)
 		(end 154.305 121.92)
@@
 	)
 	(segment
-		(start 148.59 135.89)
-		(end 142.24 142.24)
-		(width 0.5)
-		(layer "B.Cu")
-		(net 16)
-	)
-	(segment
-		(start 153.67 137.16)
-		(end 153.67 135.89)
-		(width 1)
-		(layer "B.Cu")
-		(net 16)
-	)
-	(segment
 		(start 160.02 91.44)
 		(end 160.02 115.57)
@@
 		(start 142.24 142.24)
 		(end 124.46 142.24)
-		(width 0.5)
+		(width 1)
 		(layer "B.Cu")
 		(net 16)
@@
 	)
 	(segment
-		(start 165.1 96.52)
-		(end 165.57 96.05)
+		(start 164.83 94.615)
+		(end 165.1 94.885)
 		(width 0.2)
 		(layer "F.Cu")
@@
 	)
 	(segment
-		(start 165.57 96.05)
-		(end 165.57 94.73)
+		(start 165.1 94.885)
+		(end 165.1 96.52)
 		(width 0.2)
 		(layer "F.Cu")
@@
 	)
 	(segment
-		(start 167.67 99.03)
-		(end 167.64 99.06)
-		(width 0.2)
-		(layer "B.Cu")
-		(net 41)
-	)
-	(segment
-		(start 165.1 96.52)
-		(end 165.57 96.05)
-		(width 0.2)
-		(layer "B.Cu")
-		(net 41)
-	)
-	(segment
 		(start 165.1 96.52)
 		(end 165.1 99.06)
@@
 	)
 	(segment
-		(start 165.69 92.64)
-		(end 167.67 94.62)
+		(start 167.005 99.06)
+		(end 165.1 99.06)
 		(width 0.2)
 		(layer "B.Cu")
@@
 	(segment
 		(start 165.1 92.64)
-		(end 165.69 92.64)
-		(width 0.2)
-		(layer "B.Cu")
-		(net 41)
-	)
-	(segment
-		(start 167.64 99.06)
-		(end 165.1 99.06)
+		(end 167.005 94.545)
 		(width 0.2)
 		(layer "B.Cu")
@@
 	)
 	(segment
-		(start 167.67 94.62)
-		(end 167.67 99.03)
+		(start 167.005 94.545)
+		(end 167.005 99.06)
 		(width 0.2)
 		(layer "B.Cu")
