File: ESP32-E22_V2.1.1/KiCad/esp32-e22.kicad_pcb (KiCad board)
At the start: 2 copper layers, 70 x 99 mm, 42 parts, among them J1 Conn_01x02_Socket, J10 Conn_01x02_Socket, J3 Conn_01x02_Socket, J4 Conn_01x04_Socket, J5 Conn_01x03_Socket, J6 Conn_01x04_Socket, J7 Conn_01x04_Socket, J8 SMA, J9 Conn_01x02_Socket, SW1 SW_Push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

Commit message: update
Parts:
- moved C8 2.58 mm to (115.6, 72.4)
- moved J6 1.27 mm to (124.5, 77.5)
Routing:
- net +3.3V: track 172.8 -> 174.3 mm
- net /SCL: track 106.4 -> 107.7 mm
- net /SDA: track 121.9 -> 123.2 mm
Changed lines of the file:
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@@
 	(title_block
 		(title "ESP32+E22 single sided")
-		(date "2024-10-16")
+		(date "2024-10-19")
 		(rev "V 2.1.1")
 		(comment 1 "designed by OE3WAS")
@@
 	(footprint "Connector_PinHeader_2.54mm:PinHeader_1x04_P2.54mm_Vertical"
 		(layer "F.Cu")
-		(at 123.19 77.47 180)
+		(at 124.46 77.47 180)
 		(descr "Through hole straight pin header, 1x04, 2.54mm pitch, single row")
 		(tags "Through hole pin header THT 1x04 2.54mm single row")
@@
 	(footprint "Capacitor_THT:C_Disc_D4.7mm_W2.5mm_P5.00mm"
 		(layer "F.Cu")
-		(at 115.57 74.97 -90)
+		(at 115.57 72.39 -90)
 		(descr "C, Disc series, Radial, pin pitch=5.00mm, , diameter*width=4.7*2.5mm^2, Capacitor, http://www.vishay.com/docs/45233/krseries.pdf")
 		(tags "C Disc series Radial pin pitch 5.00mm  diameter 4.7mm width 2.5mm Capacitor")
@@
 		)
 	)
+	(gr_circle
+		(center 124.46 69.85)
+		(end 124.46 70.485)
+		(stroke
+			(width 0.1)
+			(type default)
+		)
+		(fill none)
+		(layer "Dwgs.User")
+	)
+	(gr_circle
+		(center 124.46 72.39)
+		(end 123.825 72.39)
+		(stroke
+			(width 0.1)
+			(type default)
+		)
+		(fill none)
+		(layer "Dwgs.User")
+	)
+	(gr_circle
+		(center 124.46 74.93)
+		(end 123.825 74.93)
+		(stroke
+			(width 0.1)
+			(type default)
+		)
+		(fill none)
+		(layer "Dwgs.User")
+	)
+	(gr_circle
+		(center 124.46 77.47)
+		(end 123.825 77.47)
+		(stroke
+			(width 0.1)
+			(type default)
+		)
+		(fill none)
+		(layer "Dwgs.User")
+	)
+	(gr_rect
+		(start 113.03 68.58)
+		(end 125.73 78.74)
+		(stroke
+			(width 0.1)
+			(type default)
+		)
+		(fill none)
+		(layer "Dwgs.User")
+	)
 	(gr_arc
 		(start 166.57 46.93)
@@
 	)
 	(segment
+		(start 120.65 93.98)
+		(end 120.65 80.01)
+		(width 0.3)
+		(layer "F.Cu")
+		(net 2)
+	)
+	(segment
 		(start 161.29 97.79)
 		(end 162.56 99.06)
@@
 	)
 	(segment
-		(start 120.65 93.98)
-		(end 120.65 80.01)
+		(start 120.65 80.01)
+		(end 123.19 77.47)
 		(width 0.3)
 		(layer "F.Cu")
@@
 	)
 	(segment
-		(start 120.65 80.01)
-		(end 123.19 77.47)
+		(start 173.99 82.54)
+		(end 170.19 78.74)
 		(width 0.3)
 		(layer "F.Cu")
@@
 	)
 	(segment
-		(start 173.99 82.54)
-		(end 170.19 78.74)
+		(start 173.99 93.98)
+		(end 173.99 82.54)
 		(width 0.3)
 		(layer "F.Cu")
@@
 	)
 	(segment
-		(start 173.99 93.98)
-		(end 173.99 82.54)
+		(start 123.19 77.47)
+		(end 124.46 77.47)
 		(width 0.3)
 		(layer "F.Cu")
@@
 	)
 	(segment
-		(start 115.57 79.97)
-		(end 118.07 77.47)
+		(start 122.555 115.291346)
+		(end 121.563654 114.3)
 		(width 0.3)
 		(layer "B.Cu")
@@
 	)
 	(segment
-		(start 122.555 115.291346)
-		(end 121.563654 114.3)
+		(start 118.07 77.47)
+		(end 124.46 77.47)
 		(width 0.3)
 		(layer "B.Cu")
@@
 	)
 	(segment
+		(start 117.99 77.39)
+		(end 118.07 77.47)
+		(width 0.3)
+		(layer "B.Cu")
+		(net 2)
+	)
+	(segment
 		(start 118.11 101.6)
 		(end 118.11 95.25)
@@
 	)
 	(segment
+		(start 115.57 77.39)
+		(end 117.99 77.39)
+		(width 0.3)
+		(layer "B.Cu")
+		(net 2)
+	)
+	(segment
 		(start 123.19 96.52)
 		(end 124.46 96.52)
@@
 		(net 2)
 	)
-	(segment
-		(start 118.07 77.47)
-		(end 123.19 77.47)
-		(width 0.3)
-		(layer "B.Cu")
-		(net 2)
-	)
 	(via
 		(at 155.87 99.73)
@@
 	)
 	(segment
-		(start 135.89 109.22)
-		(end 127 100.33)
+		(start 122.555 100.33)
+		(end 118.11 95.885)
 		(width 0.3)
 		(layer "F.Cu")
@@
 	)
 	(segment
-		(start 172.72 104.775)
-		(end 170.18 107.315)
+		(start 149.86 109.22)
+		(end 135.89 109.22)
 		(width 0.3)
 		(layer "F.Cu")
@@
 	)
 	(segment
-		(start 168.275 109.22)
+		(start 172.72 104.775)
 		(end 170.18 107.315)
 		(width 0.3)
@@
 	)
 	(segment
-		(start 149.86 109.22)
-		(end 135.89 109.22)
+		(start 127 100.33)
+		(end 122.555 100.33)
 		(width 0.3)
 		(layer "F.Cu")
@@
 	)
 	(segment
-		(start 118.11 95.885)
-		(end 118.11 74.93)
+		(start 168.275 109.22)
+		(end 170.18 107.315)
 		(width 0.3)
 		(layer "F.Cu")
@@
 	)
 	(segment
-		(start 122.555 100.33)
-		(end 118.11 95.885)
+		(start 135.89 109.22)
+		(end 127 100.33)
 		(width 0.3)
 		(layer "F.Cu")
@@
 	)
 	(segment
-		(start 118.11 74.93)
-		(end 123.19 69.85)
+		(start 118.11 95.885)
+		(end 118.11 74.93)
 		(width 0.3)
 		(layer "F.Cu")
@@
 	)
 	(segment
-		(start 127 100.33)
-		(end 122.555 100.33)
+		(start 118.11 74.93)
+		(end 123.19 69.85)
+		(width 0.3)
+		(layer "F.Cu")
+		(net 5)
+	)
+	(segment
+		(start 123.19 69.85)
+		(end 124.46 69.85)
 		(width 0.3)
 		(layer "F.Cu")
@@
 	)
 	(segment
-		(start 121.92 97.79)
-		(end 119.38 95.25)
+		(start 119.38 95.25)
+		(end 119.38 76.2)
 		(width 0.3)
 		(layer "F.Cu")
@@
 	)
 	(segment
-		(start 149.86 101.6)
-		(end 130.81 101.6)
+		(start 130.81 101.6)
+		(end 127 97.79)
 		(width 0.3)
 		(layer "F.Cu")
@@
 	)
 	(segment
-		(start 167.64 101.6)
-		(end 170.18 104.14)
+		(start 149.86 101.6)
+		(end 130.81 101.6)
 		(width 0.3)
 		(layer "F.Cu")
@@
 	)
 	(segment
-		(start 119.38 95.25)
-		(end 119.38 76.2)
+		(start 167.64 101.6)
+		(end 170.18 104.14)
 		(width 0.3)
 		(layer "F.Cu")
@@
 	)
 	(segment
-		(start 130.81 101.6)
-		(end 127 97.79)
+		(start 121.92 97.79)
+		(end 119.38 95.25)
+		(width 0.3)
+		(layer "F.Cu")
+		(net 6)
+	)
+	(segment
+		(start 123.19 72.39)
+		(end 124.46 72.39)
 		(width 0.3)
 		(layer "F.Cu")

Commit message: update to V2.1.1-α2
Parts:
- J6: footprint Connector_PinHeader_2.54mm:PinHeader_1x04_P2.54mm_Vertical -> Connector_PinSocket_2.54mm:PinSocket_1x04_P2.54mm_Vertical
Changed lines of the file:
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@@
 		)
 	)
-	(footprint "Connector_PinHeader_2.54mm:PinHeader_1x04_P2.54mm_Vertical"
+	(footprint "Connector_PinSocket_2.54mm:PinSocket_1x04_P2.54mm_Vertical"
 		(layer "F.Cu")
 		(at 124.46 77.47 180)
-		(descr "Through hole straight pin header, 1x04, 2.54mm pitch, single row")
-		(tags "Through hole pin header THT 1x04 2.54mm single row")
+		(descr "Through hole straight socket strip, 1x04, 2.54mm pitch, single row (from Kicad 4.0.7), script generated")
+		(tags "Through hole socket strip THT 1x04 2.54mm single row")
 		(property "Reference" "J6"
-			(at 0 -2.33 0)
+			(at 0 -2.77 180)
 			(layer "F.SilkS")
 			(effects
@@
 		)
 		(property "Value" "Conn_01x04_Socket"
-			(at 0 9.95 0)
-			(layer "F.Fab")
-			(effects
-				(font
-					(size 1 1)
-					(thickness 0.15)
-				)
-			)
-		)
-		(property "Footprint" "Connector_PinHeader_2.54mm:PinHeader_1x04_P2.54mm_Vertical"
+			(at 0 10.39 180)
+			(layer "F.Fab")
+			(effects
+				(font
+					(size 1 1)
+					(thickness 0.15)
+				)
+			)
+		)
+		(property "Footprint" "Connector_PinSocket_2.54mm:PinSocket_1x04_P2.54mm_Vertical"
 			(at 0 0 180)
 			(unlocked yes)
@@
 		)
 		(fp_line
+			(start 1.33 -1.33)
+			(end 1.33 0)
+			(stroke
+				(width 0.12)
+				(type solid)
+			)
+			(layer "F.SilkS")
+		)
+		(fp_line
+			(start 0 -1.33)
+			(end 1.33 -1.33)
+			(stroke
+				(width 0.12)
+				(type solid)
+			)
+			(layer "F.SilkS")
+		)
+		(fp_line
 			(start -1.33 8.95)
 			(end 1.33 8.95)
@@
 		)
 		(fp_line
-			(start -1.33 0)
-			(end -1.33 -1.33)
-			(stroke
-				(width 0.12)
-				(type solid)
-			)
-			(layer "F.SilkS")
-		)
-		(fp_line
-			(start -1.33 -1.33)
-			(end 0 -1.33)
-			(stroke
-				(width 0.12)
-				(type solid)
-			)
-			(layer "F.SilkS")
-		)
-		(fp_line
-			(start 1.8 9.4)
-			(end 1.8 -1.8)
-			(stroke
-				(width 0.05)
-				(type solid)
-			)
-			(layer "F.CrtYd")
-		)
-		(fp_line
-			(start 1.8 -1.8)
+			(start 1.75 9.4)
+			(end -1.8 9.4)
+			(stroke
+				(width 0.05)
+				(type solid)
+			)
+			(layer "F.CrtYd")
+		)
+		(fp_line
+			(start 1.75 -1.8)
+			(end 1.75 9.4)
+			(stroke
+				(width 0.05)
+				(type solid)
+			)
+			(layer "F.CrtYd")
+		)
+		(fp_line
+			(start -1.8 9.4)
 			(end -1.8 -1.8)
 			(stroke
@@
 		)
 		(fp_line
-			(start -1.8 9.4)
-			(end 1.8 9.4)
-			(stroke
-				(width 0.05)
-				(type solid)
-			)
-			(layer "F.CrtYd")
-		)
-		(fp_line
 			(start -1.8 -1.8)
-			(end -1.8 9.4)
+			(end 1.75 -1.8)
 			(stroke
 				(width 0.05)
@@
 		)
 		(fp_line
-			(start 1.27 -1.27)
+			(start 1.27 -0.635)
 			(end 1.27 8.89)
 			(stroke
@@
 		)
 		(fp_line
-			(start -0.635 -1.27)
-			(end 1.27 -1.27)
+			(start 0.635 -1.27)
+			(end 1.27 -0.635)
 			(stroke
 				(width 0.1)
@@
 		(fp_line
 			(start -1.27 8.89)
-			(end -1.27 -0.635)
-			(stroke
-				(width 0.1)
-				(type solid)
-			)
-			(layer "F.Fab")
-		)
-		(fp_line
-			(start -1.27 -0.635)
-			(end -0.635 -1.27)
+			(end -1.27 -1.27)
+			(stroke
+				(width 0.1)
+				(type solid)
+			)
+			(layer "F.Fab")
+		)
+		(fp_line
+			(start -1.27 -1.27)
+			(end 0.635 -1.27)
 			(stroke
 				(width 0.1)
@@
 		)
 		(fp_text user "${REFERENCE}"
-			(at 0 3.81 90)
+			(at 0 3.81 -90)
 			(layer "F.Fab")
 			(effects
@@
 			(pintype "passive")
 		)
-		(model "${KICAD8_3DMODEL_DIR}/Connector_PinHeader_2.54mm.3dshapes/PinHeader_1x04_P2.54mm_Vertical.wrl"
+		(model "${KICAD8_3DMODEL_DIR}/Connector_PinSocket_2.54mm.3dshapes/PinSocket_1x04_P2.54mm_Vertical.wrl"
 			(offset
 				(xyz 0 0 0)

Commit message: update
Parts:
- J3: value Conn_01x02_Socket -> Screw_Terminal_01x02
- J7: footprint Connector_PinHeader_2.54mm:PinHeader_1x04_P2.54mm_Vertical -> Connector_PinSocket_2.54mm:PinSocket_1x04_P2.54mm_Vertical
- moved J3 0.31 mm to (171.4, 128.6)

Commit message: update
Parts:
- J7: value Conn_01x04_Socket -> Conn_01x05_Socket; footprint Connector_PinSocket_2.54mm:PinSocket_1x04_P2.54mm_Vertical -> Connector_PinSocket_2.54mm:PinSocket_1x05_P2.54mm_Vertical
- moved J7 6.47 mm to (176.5, 80.0), turned to 180 degrees
- moved C7 5.19 mm to (171.4, 69.9), turned to -90 degrees
- moved J10 0.64 mm to (116.2, 128.3)
Routing:
- net +3.3V: track 174.3 -> 185.5 mm
- net /SDA: track 123.2 -> 129.1 mm
- net /SCL: track 107.7 -> 110.5 mm

Commit message: Update esp32-e22.kicad_pcb
Parts:
- added REF**: MountingHole_2.1mm, MountingHole:MountingHole_2.1mm, F.Cu at (176.5, 68.6)
- moved J7 3.81 mm to (176.5, 83.8)
- moved C7 3.77 mm to (171.4, 73.7)
Routing:
- net +3.3V: track 185.5 -> 181.8 mm
- net /SCL: track 110.5 -> 107.5 mm
- net /SDA: track 129.1 -> 126.7 mm
Changed lines of the file:
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@@
 	(footprint "Connector_PinSocket_2.54mm:PinSocket_1x05_P2.54mm_Vertical"
 		(layer "F.Cu")
-		(at 176.53 80.01 180)
+		(at 176.53 83.82 180)
 		(descr "Through hole straight socket strip, 1x05, 2.54mm pitch, single row (from Kicad 4.0.7), script generated")
 		(tags "Through hole socket strip THT 1x05 2.54mm single row")
 		(property "Reference" "J7"
-			(at 0 13.335 360)
+			(at 0 -3.81 0)
 			(layer "F.SilkS")
 			(effects
@@
 		)
 		(property "Value" "Conn_01x05_Socket"
-			(at 0 12.93 360)
+			(at 0 12.93 0)
 			(layer "F.Fab")
 			(effects
@@
 		)
 	)
+	(footprint "MountingHole:MountingHole_2.1mm"
+		(layer "F.Cu")
+		(at 176.53 68.58)
+		(descr "Mounting Hole 2.1mm, no annular")
+		(tags "mounting hole 2.1mm no annular")
+		(property "Reference" "REF**"
+			(at 0 -3.2 0)
+			(layer "F.SilkS")
+			(effects
+				(font
+					(size 1 1)
+					(thickness 0.15)
+				)
+			)
+		)
+		(property "Value" "MountingHole_2.1mm"
+			(at 0 3.2 0)
+			(layer "F.Fab")
+			(effects
+				(font
+					(size 1 1)
+					(thickness 0.15)
+				)
+			)
+		)
+		(property "Footprint" "MountingHole:MountingHole_2.1mm"
+			(at 0 0 0)
+			(unlocked yes)
+			(layer "F.Fab")
+			(hide yes)
+			(effects
+				(font
+					(size 1.27 1.27)
+					(thickness 0.15)
+				)
+			)
+		)
+		(property "Datasheet" ""
+			(at 0 0 0)
+			(unlocked yes)
+			(layer "F.Fab")
+			(hide yes)
+			(effects
+				(font
+					(size 1.27 1.27)
+					(thickness 0.15)
+				)
+			)
+		)
+		(property "Description" ""
+			(at 0 0 0)
+			(unlocked yes)
+			(layer "F.Fab")
+			(hide yes)
+			(effects
+				(font
+					(size 1.27 1.27)
+					(thickness 0.15)
+				)
+			)
+		)
+		(attr exclude_from_pos_files exclude_from_bom)
+		(fp_circle
+			(center 0 0)
+			(end 2.1 0)
+			(stroke
+				(width 0.15)
+				(type solid)
+			)
+			(fill none)
+			(layer "Cmts.User")
+		)
+		(fp_circle
+			(center 0 0)
+			(end 2.35 0)
+			(stroke
+				(width 0.05)
+				(type solid)
+			)
+			(fill none)
+			(layer "F.CrtYd")
+		)
+		(fp_text user "${REFERENCE}"
+			(at 0 0 0)
+			(layer "F.Fab")
+			(effects
+				(font
+					(size 1 1)
+					(thickness 0.15)
+				)
+			)
+		)
+		(pad "" np_thru_hole circle
+			(at 0 0)
+			(size 2.1 2.1)
+			(drill 2.1)
+			(layers "*.Cu" "*.Mask")
+		)
+	)
 	(footprint "Capacitor_THT:CP_Radial_D5.0mm_P2.50mm"
 		(layer "F.Cu")
@@
 	(footprint "Capacitor_THT:C_Disc_D4.7mm_W2.5mm_P5.00mm"
 		(layer "F.Cu")
-		(at 171.45 69.89 -90)
+		(at 171.45 73.66 -90)
 		(descr "C, Disc series, Radial, pin pitch=5.00mm, , diameter*width=4.7*2.5mm^2, Capacitor, http://www.vishay.com/docs/45233/krseries.pdf")
 		(tags "C Disc series Radial pin pitch 5.00mm  diameter 4.7mm width 2.5mm Capacitor")
@@
 	)
 	(segment
-		(start 127 96.52)
-		(end 128.27 97.79)
-		(width 0.3)
-		(layer "F.Cu")
-		(net 2)
-	)
-	(segment
-		(start 124.46 96.52)
-		(end 127 96.52)
+		(start 173.99 93.98)
+		(end 173.99 76.2)
 		(width 0.3)
 		(layer "F.Cu")
@@
 	)
 	(segment
-		(start 173.99 80.01)
-		(end 173.99 72.43)
+		(start 173.99 76.2)
+		(end 171.45 73.66)
 		(width 0.3)
 		(layer "F.Cu")
@@
 	)
 	(segment
-		(start 173.99 80.01)
-		(end 176.53 80.01)
+		(start 127 96.52)
+		(end 128.27 97.79)
 		(width 0.3)
 		(layer "F.Cu")
@@
 	)
 	(segment
-		(start 128.27 97.79)
-		(end 161.29 97.79)
+		(start 124.46 96.52)
+		(end 127 96.52)
 		(width 0.3)
 		(layer "F.Cu")
@@
 	)
 	(segment
-		(start 173.99 93.98)
-		(end 173.99 80.01)
+		(start 173.99 83.82)
+		(end 176.53 83.82)
 		(width 0.3)
 		(layer "F.Cu")
@@
 	)
 	(segment
-		(start 173.99 72.43)
-		(end 171.45 69.89)
+		(start 128.27 97.79)
+		(end 161.29 97.79)
 		(width 0.3)
 		(layer "F.Cu")
@@
 	)
 	(segment
-		(start 176.53 69.85)
-		(end 175.26 69.85)
-		(width 0.3)
-		(layer "B.Cu")
-		(net 2)
-	)
-	(segment
 		(start 118.11 95.25)
 		(end 119.38 95.25)
@@
 	)
 	(segment
-		(start 175.22 69.89)
-		(end 171.45 69.89)
-		(width 0.3)
-		(layer "B.Cu")
-		(net 2)
-	)
-	(segment
 		(start 118.11 101.6)
 		(end 118.11 95.25)
@@
 	)
 	(segment
+		(start 176.53 73.66)
+		(end 171.45 73.66)
+		(width 0.3)
+		(layer "B.Cu")
+		(net 2)
+	)
+	(segment
 		(start 116.84 114.3)
 		(end 115.57 113.03)
@@
 	)
 	(segment
-		(start 175.26 69.85)
-		(end 175.22 69.89)
-		(width 0.3)
-		(layer "B.Cu")
-		(net 2)
-	)
-	(segment
 		(start 122.555 130.165)
 		(end 122.555 115.291346)
@@
 	)
 	(segment
-		(start 178.435 74.295)
-		(end 176.53 72.39)
+		(start 178.435 86.995)
+		(end 178.435 78.105)
 		(width 0.3)
 		(layer "B.Cu")
@@
 	)
 	(segment
-		(start 178.435 84.455)
-		(end 178.435 74.295)
+		(start 172.79 92.64)
+		(end 178.435 86.995)
 		(width 0.3)
 		(layer "B.Cu")
@@
 	)
 	(segment
-		(start 170.18 92.64)
-		(end 170.25 92.64)
+		(start 178.435 78.105)
+		(end 176.53 76.2)
 		(width 0.3)
 		(layer "B.Cu")
@@
 	)
 	(segment
-		(start 170.25 92.64)
-		(end 178.435 84.455)
+		(start 170.18 92.64)
+		(end 172.79 92.64)
 		(width 0.3)
 		(layer "B.Cu")
@@
 	)
 	(segment
+		(start 173.99 80.01)
+		(end 175.26 78.74)
+		(width 0.3)
+		(layer "B.Cu")
+		(net 6)
+	)
+	(segment
 		(start 167.64 92.64)
 		(end 173.99 86.29)
@@
 	(segment
 		(start 173.99 86.29)
-		(end 173.99 77.47)
+		(end 173.99 80.01)
 		(width 0.3)
 		(layer "B.Cu")
@@
 	)
 	(segment
-		(start 173.99 77.47)
-		(end 176.53 74.93)
+		(start 175.26 78.74)
+		(end 176.53 78.74)
 		(width 0.3)
 		(layer "B.Cu")

Commit message: mask update
Routing:
- net GND: vias 2 -> 27
Changed lines of the file:
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@@
+	)
+	(via
+		(at 143.51 67.31)
+		(size 0.6)
+		(drill 0.3)
+		(layers "F.Cu" "B.Cu")
+		(free yes)
+		(net 3)
+	)
+	(via
+		(at 140.97 67.31)
+		(size 0.6)
+		(drill 0.3)
+		(layers "F.Cu" "B.Cu")
+		(free yes)
+		(net 3)
+	)
+	(via
+		(at 138.43 74.93)
+		(size 0.6)
+		(drill 0.3)
+		(layers "F.Cu" "B.Cu")
+		(free yes)
+		(net 3)
+	)
+	(via
+		(at 138.43 72.39)
+		(size 0.6)
+		(drill 0.3)
+		(layers "F.Cu" "B.Cu")
+		(free yes)
+		(net 3)
+	)
+	(via
+		(at 143.51 72.39)
+		(size 0.6)
+		(drill 0.3)
+		(layers "F.Cu" "B.Cu")
+		(free yes)
+		(net 3)
+	)
+	(via
+		(at 143.51 74.93)
+		(size 0.6)
+		(drill 0.3)
+		(layers "F.Cu" "B.Cu")
+		(free yes)
+		(net 3)
+	)
+	(via
+		(at 138.43 69.85)
+		(size 0.6)
+		(drill 0.3)
+		(layers "F.Cu" "B.Cu")
+		(free yes)
+		(net 3)
 	)
 	(via
@@
 	(via
 		(at 155.97 105.43)
+		(size 0.6)
+		(drill 0.3)
+		(layers "F.Cu" "B.Cu")
+		(free yes)
+		(net 3)
+	)
+	(via
+		(at 143.51 64.77)
+		(size 0.6)
+		(drill 0.3)
+		(layers "F.Cu" "B.Cu")
+		(free yes)
+		(net 3)
+	)
+	(via
+		(at 140.97 69.85)
+		(size 0.6)
+		(drill 0.3)
+		(layers "F.Cu" "B.Cu")
+		(free yes)
+		(net 3)
+	)
+	(via
+		(at 133.35 69.85)
+		(size 0.6)
+		(drill 0.3)
+		(layers "F.Cu" "B.Cu")
+		(free yes)
+		(net 3)
+	)
+	(via
+		(at 133.35 67.31)
+		(size 0.6)
+		(drill 0.3)
+		(layers "F.Cu" "B.Cu")
+		(free yes)
+		(net 3)
+	)
+	(via
+		(at 133.35 64.77)
+		(size 0.6)
+		(drill 0.3)
+		(layers "F.Cu" "B.Cu")
+		(free yes)
+		(net 3)
+	)
+	(via
+		(at 138.43 67.31)
+		(size 0.6)
+		(drill 0.3)
+		(layers "F.Cu" "B.Cu")
+		(free yes)
+		(net 3)
+	)
+	(via
+		(at 140.97 64.77)
+		(size 0.6)
+		(drill 0.3)
+		(layers "F.Cu" "B.Cu")
+		(free yes)
+		(net 3)
+	)
+	(via
+		(at 143.51 69.85)
+		(size 0.6)
+		(drill 0.3)
+		(layers "F.Cu" "B.Cu")
+		(free yes)
+		(net 3)
+	)
+	(via
+		(at 135.89 67.31)
+		(size 0.6)
+		(drill 0.3)
+		(layers "F.Cu" "B.Cu")
+		(free yes)
+		(net 3)
+	)
+	(via
+		(at 140.97 74.93)
+		(size 0.6)
+		(drill 0.3)
+		(layers "F.Cu" "B.Cu")
+		(free yes)
+		(net 3)
+	)
+	(via
+		(at 135.89 64.77)
+		(size 0.6)
+		(drill 0.3)
+		(layers "F.Cu" "B.Cu")
+		(free yes)
+		(net 3)
+	)
+	(via
+		(at 135.89 74.93)
+		(size 0.6)
+		(drill 0.3)
+		(layers "F.Cu" "B.Cu")
+		(free yes)
+		(net 3)
+	)
+	(via
+		(at 138.43 64.77)
+		(size 0.6)
+		(drill 0.3)
+		(layers "F.Cu" "B.Cu")
+		(free yes)
+		(net 3)
+	)
+	(via
+		(at 140.97 72.39)
+		(size 0.6)
+		(drill 0.3)
+		(layers "F.Cu" "B.Cu")
+		(free yes)
+		(net 3)
+	)
+	(via
+		(at 135.89 69.85)
+		(size 0.6)
+		(drill 0.3)
+		(layers "F.Cu" "B.Cu")
+		(free yes)
+		(net 3)
+	)
+	(via
+		(at 133.35 72.39)
+		(size 0.6)
+		(drill 0.3)
+		(layers "F.Cu" "B.Cu")
+		(free yes)
+		(net 3)
+	)
+	(via
+		(at 133.35 74.93)
+		(size 0.6)
+		(drill 0.3)
+		(layers "F.Cu" "B.Cu")
+		(free yes)
+		(net 3)
+	)
+	(via
+		(at 135.89 72.39)
 		(size 0.6)
 		(drill 0.3)
@@
 			)
 		)
+	)
+	(zone
+		(net 0)
+		(net_name "")
+		(layers "*.Mask")
+		(hatch full 0.5)
+		(connect_pads
+			(clearance 0.5)
+		)
+		(min_thickness 0.25)
+		(filled_areas_thickness no)
+		(fill yes
+			(thermal_gap 0.5)
+			(thermal_bridge_width 0.5)
+		)
+		(polygon
+			(pts
+				(xy 142.24 54.61) (xy 167.64 54.61) (xy 167.64 48.26) (xy 142.24 48.26)
+			)
+		)
+	)
+	(zone
+		(net 0)
+		(net_name "")
+		(layer "F.Mask")
+		(hatch edge 0.5)
+		(connect_pads
+			(clearance 0.5)
+		)
+		(min_thickness 0.25)
+		(filled_areas_thickness no)
+		(fill yes
+			(thermal_gap 0.5)
+			(thermal_bridge_width 0.5)
+		)
+		(polygon
+			(pts
+				(xy 132.08 76.2) (xy 144.78 76.2) (xy 144.78 63.5) (xy 132.08 63.5)
+			)
+		)

Commit message: PCB V2.1.1-α3
Parts:
- moved C8 5.08 mm to (120.7, 72.4)
- moved C2 0.64 mm to (125.1, 88.9)
Routing:
- net +3.3V: track 181.8 -> 175.7 mm
- net /SDA: track 126.7 -> 128.8 mm
- net /SCL: track 107.5 -> 108.0 mm
- net GND: vias 27 -> 41

Commit message: SCH & PCB α5
Parts:
- added D5: 1N4004, Diode_THT:D_DO-41_SOD81_P5.08mm_Vertical_KathodeUp, F.Cu at (166.4, 124.9)
- added U4: Mini_DC-DC_12-24V_adjustable, KiCad:HW-613, B.Cu at (158.1, 141.6)
- D1: footprint Diode_THT:D_DO-41_SOD81_P7.62mm_Horizontal -> Diode_THT:D_DO-41_SOD81_P5.08mm_Vertical_KathodeUp
- D2, R3, R4: moved to B.Cu
- F1: value 5A -> 2A
- moved R3 20.7 mm to (155.6, 144.1)
- moved D1 18.1 mm to (166.4, 138.6), turned to 90 degrees
- moved R4 14.5 mm to (155.6, 141.0)
- moved C5 14.2 mm to (166.4, 143.5), turned to 0 degrees
- moved C6 12.7 mm to (167.0, 121.9)
- moved D2 9.44 mm to (170.2, 116.2), turned to 180 degrees
- moved D3 4.49 mm to (161.9, 122.6)
- moved J2 3.86 mm to (158.1, 130.2)
- moved D4 3.17 mm to (172.7, 111.1)
- moved J3 0.64 mm to (172.1, 128.6)
- moved R7 0.64 mm to (162.6, 103.5)
- moved R6 0.63 mm to (162.6, 106.7)
- moved F1 0.34 mm to (177.5, 120.0)
Connections:
- F1 pad 1: Net-(J3-Pin_1) -> Net-(J3-Pin_2)
- F1 pad 2: Net-(D2-A) -> Net-(D5-K)
- J3 pad 1: Net-(J3-Pin_1) -> GND
- J3 pad 2: GND -> Net-(J3-Pin_2)
Routing:
- net Net-(D5-K): track 0.00 -> 20.0 mm
- net Net-(J3-Pin_1): track 10.9 -> 0.00 mm
- net Net-(D1-A): track 5.87 -> 14.6 mm
- net Net-(J3-Pin_2): track 0.00 -> 8.70 mm
- net +5V: track 132.8 -> 140.6 mm
- net +3.3V: track 175.7 -> 168.2 mm
- net Net-(J2-CC2): track 8.56 -> 15.5 mm
- net Net-(J2-CC1): track 4.34 -> 11.3 mm
- net /OneWire: track 28.2 -> 22.4 mm
- net Net-(D2-A): track 3.44 -> 4.23 mm
- net GND: track 0.00 -> 0.64 mm
- net /GPS_TX: track 39.6 -> 40.1 mm
- net Net-(J1-Pin_1): track 11.2 -> 11.7 mm
