File: ESP32-E22_V2.1.1/KiCad/esp32-e22.kicad_pcb (KiCad board)
At the start: 2 copper layers, 70 x 99 mm, 45 parts, among them J1 Conn_01x02_Socket, J10 Conn_01x02_Socket, J3 Screw_Terminal_01x02, J4 Conn_01x04_Socket, J5 Conn_01x03_Socket, J6 Conn_01x04_Socket, J7 Conn_01x05_Socket, J8 SMA, J9 Conn_01x02_Socket, SW1 SW_Push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

Commit message: update
Parts:
- moved C3 2.29 mm to (164.5, 88.9), turned to 90 degrees
- moved D1 1.05 mm to (166.4, 139.7)
- moved D5 0.85 mm to (166.4, 125.7)
- moved C6 0.06 mm to (167.0, 121.9)
Routing:
- net Net-(D5-K): track 20.0 -> 20.7 mm
Other:
- board text added: "+"
- board text added: "-"

Commit message: update PCB
Parts:
- moved J5 6.35 mm to (115.6, 88.9)
Routing:
- net /OneWire: track 22.4 -> 26.5 mm
- net +3.3V: track 168.2 -> 167.0 mm
Other:
- outline, holes or cut-outs redrawn
- board text added: "ESP32-E22 V2.1.1 by OE3WAS"
- board text removed: "ESP32-E22 V2.1.1 designed by OE3WAS"
Changed lines of the file:
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@@
 	(footprint "Connector_PinHeader_2.54mm:PinHeader_1x03_P2.54mm_Vertical"
 		(layer "F.Cu")
-		(at 115.57 95.25)
+		(at 115.57 88.9)
 		(descr "Through hole straight pin header, 1x03, 2.54mm pitch, single row")
 		(tags "Through hole pin header THT 1x03 2.54mm single row")
@@
 		(layer "Dwgs.User")
 	)
-	(gr_arc
-		(start 166.57 46.93)
-		(mid 169.398427 48.101573)
-		(end 170.57 50.93)
+	(gr_line
+		(start 170.57 55.93)
+		(end 144.57 55.93)
 		(stroke
 			(width 0.05)
@@
 		(layer "Edge.Cuts")
 	)
+	(gr_line
+		(start 144.57 55.93)
+		(end 144.57 46.93)
+		(stroke
+			(width 0.05)
+			(type default)
+		)
+		(layer "Edge.Cuts")
+	)
 	(gr_arc
 		(start 129.57 50.93)
@@
 	)
 	(gr_line
-		(start 166.57 46.93)
+		(start 144.57 46.93)
 		(end 133.57 46.93)
 		(stroke
@@
 		(layer "Edge.Cuts")
 	)
-	(gr_line
-		(start 170.57 55.93)
-		(end 170.57 50.93)
-		(stroke
-			(width 0.05)
-			(type default)
-		)
-		(layer "Edge.Cuts")
-	)
-	(gr_text "ESP32-E22 V2.1.1\ndesigned by OE3WAS"
-		(at 143.51 53.34 0)
+	(gr_text "ESP32-E22\nV2.1.1\nby OE3WAS"
+		(at 122.555 62.865 0)
 		(layer "F.Cu")
 		(effects
 			(font
-				(size 1.5 1.5)
-				(thickness 0.3)
+				(size 1.1 1.1)
+				(thickness 0.2)
 				(bold yes)
 			)
-			(justify left bottom)
+			(justify bottom)
 		)
 	)
-	(gr_text "ESP32-E22 V2.1.1\ndesigned by OE3WAS"
-		(at 166.37 53.34 0)
+	(gr_text "ESP32-E22\nV2.1.1\nby OE3WAS"
+		(at 122.555 62.865 0)
 		(layer "B.Cu")
 		(effects
 			(font
-				(size 1.5 1.5)
-				(thickness 0.3)
+				(size 1.1 1.1)
+				(thickness 0.2)
 				(bold yes)
 			)
-			(justify left bottom mirror)
+			(justify bottom mirror)
 		)
 	)
@@
 		(layer "User.9")
 		(pts
-			(xy 170.57 53.43) (xy 129.57 53.43)
+			(xy 129.57 51.930001) (xy 144.57 51.930001)
 		)
-		(height 9.499999)
-		(gr_text "41,0000 mm"
-			(at 145.07 42.780001 0)
+		(height -7.000001)
+		(gr_text "15,0000 mm"
+			(at 137.07 43.78 0)
 			(layer "User.9")
 			(effects
@@
 			(thickness 0.1)
 			(arrow_length 1.27)
-			(text_position_mode 2)
+			(text_position_mode 0)
 			(extension_height 0.58642)
 			(extension_offset 0.5) keep_text_aligned)
@@
 	)
 	(segment
-		(start 162.56 96.52)
-		(end 162.56 92.64)
+		(start 116.84 88.9)
+		(end 120.65 85.09)
 		(width 0.3)
 		(layer "B.Cu")
@@
 	)
 	(segment
-		(start 118.745 111.76)
-		(end 118.745 95.25)
+		(start 162.56 96.52)
+		(end 162.56 92.64)
 		(width 0.3)
 		(layer "B.Cu")
@@
 	)
 	(segment
-		(start 118.11 95.25)
-		(end 119.38 95.25)
+		(start 118.745 111.76)
+		(end 118.745 95.25)
 		(width 0.3)
 		(layer "B.Cu")
@@
 	)
 	(segment
-		(start 119.38 95.25)
-		(end 120.65 93.98)
+		(start 116.84 88.9)
+		(end 115.57 88.9)
 		(width 0.3)
 		(layer "B.Cu")
@@
 	)
 	(segment
-		(start 118.11 95.25)
-		(end 115.57 95.25)
+		(start 120.65 93.98)
+		(end 120.65 92.71)
 		(width 0.3)
 		(layer "B.Cu")
@@
 	)
 	(segment
+		(start 120.65 92.71)
+		(end 116.84 88.9)
+		(width 0.3)
+		(layer "B.Cu")
+		(net 2)
+	)
+	(segment
 		(start 162.56 99.06)
 		(end 162.56 106.68)
@@
 	)
 	(segment
-		(start 120.65 93.98)
+		(start 120.65 85.09)
 		(end 120.65 77.39)
 		(width 0.3)
@@
 	)
 	(segment
-		(start 120.65 101.6)
-		(end 122.555 103.505)
+		(start 115.57 96.52)
+		(end 120.65 101.6)
 		(width 0.3)
 		(layer "F.Cu")
@@
 	)
 	(segment
-		(start 115.57 100.33)
-		(end 119.38 100.33)
+		(start 120.65 101.6)
+		(end 122.555 103.505)
 		(width 0.3)
 		(layer "F.Cu")
@@
 	)
 	(segment
-		(start 122.555 114.935)
-		(end 124.46 116.84)
+		(start 115.57 93.98)
+		(end 115.57 96.52)
 		(width 0.3)
 		(layer "F.Cu")
@@
 	)
 	(segment
-		(start 119.38 100.33)
-		(end 120.65 101.6)
+		(start 122.555 114.935)
+		(end 124.46 116.84)
 		(width 0.3)
 		(layer "F.Cu")
@@
 		(polygon
 			(pts
-				(xy 142.24 54.61) (xy 167.64 54.61) (xy 167.64 48.26) (xy 142.24 48.26)
+				(xy 117.475 63.5) (xy 128.27 63.5) (xy 128.27 57.15) (xy 117.475 57.15)
 			)
 		)
