File: ESP32-E22_V2.1.1/KiCad/esp32-e22.kicad_pcb (KiCad board)
At the start: 2 copper layers, 70 x 99 mm, 45 parts, among them J1 Conn_01x02_Socket, J10 Conn_01x02_Socket, J3 Screw_Terminal_01x02, J4 Conn_01x04_Socket, J5 Conn_01x03_Socket, J6 Conn_01x04_Socket, J7 Conn_01x05_Socket, J8 SMA, J9 Conn_01x02_Socket, SW1 SW_Push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

Commit message: update PCB V2.1.1 BETA
Parts:
- moved C2 1.27 mm to (125.1, 87.6)
- moved J5 1.27 mm to (115.6, 87.6)
- moved C7 1.27 mm to (170.2, 73.7)
Routing:
- net +3.3V: track 167.0 -> 170.6 mm
- net Net-(U1-CHIP_PU): track 13.5 -> 14.8 mm
- net /OneWire: track 26.5 -> 27.8 mm
Other:
- board text added: "1W"
- board text added: "3,3V"
- board text added: "3V3"
- board text added: "GND"
- board text added: "GPS"
- board text added: "I²C"
- board text added: "RX"
- board text added: "SCL"
- board text added: "SDA"
- board text added: "TX"

Commit message: update PCB
Routing:
- net Net-(D5-K): track 20.7 -> 22.0 mm
- net +3.3V: track 170.6 -> 171.7 mm
- net /E22_NSS: track 66.9 -> 68.0 mm
- net /E22_SCK: track 63.3 -> 63.9 mm
- net GND: vias 41 -> 42
Other:
- outline, holes or cut-outs redrawn
