File: ESP32-E22_V2.1.1/KiCad/esp32-e22.kicad_sch (KiCad schematic)
At the start: 42 parts, among them J1 Conn_01x02_Socket, J10 Conn_01x02_Socket, J3 Conn_01x02_Socket, J4 Conn_01x04_Socket, J5 Conn_01x03_Socket, J6 Conn_01x04_Socket, J7 Conn_01x04_Socket, J8 SMA, J9 Conn_01x02_Socket, SW1 SW_Push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

Commit message: update to V2.1.1-α2
Parts:
- J6: footprint Connector_PinHeader_2.54mm:PinHeader_1x04_P2.54mm_Vertical -> Connector_PinSocket_2.54mm:PinSocket_1x04_P2.54mm_Vertical
Changed lines of the file:
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@@
 			)
 		)
-		(property "Footprint" "Connector_PinHeader_2.54mm:PinHeader_1x04_P2.54mm_Vertical"
+		(property "Footprint" "Connector_PinSocket_2.54mm:PinSocket_1x04_P2.54mm_Vertical"
 			(at 190.5 78.74 0)
 			(effects

Commit message: update
Parts:
- removed J3: Conn_01x02_Socket, TerminalBlock_Phoenix:TerminalBlock_Phoenix_MKDS-1,5-2-5.08_1x02_P5.08mm_Horizontal, symbol Connector:Conn_01x02_Socket
- added J3: Screw_Terminal_01x02, TerminalBlock_Phoenix:TerminalBlock_Phoenix_MKDS-1,5-2-5.08_1x02_P5.08mm_Horizontal, symbol Connector:Screw_Terminal_01x02
- J7: footprint Connector_PinHeader_2.54mm:PinHeader_1x04_P2.54mm_Vertical -> Connector_PinSocket_2.54mm:PinSocket_1x04_P2.54mm_Vertical
Connections:
- net GND: now also J3.2 (Pin_2)
- net at F1.1: now also J3.1 (Pin_1)
Changed lines of the file:
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@@
 	(title_block
 		(title "ESP32 - E22 Board")
-		(date "2024-10-16")
+		(date "2024-10-20")
 		(rev "V2.1.1")
 		(company "DK9BT / OE3WAS")
@@
 	(wire
 		(pts
-			(xy 64.77 162.56) (xy 73.66 162.56)
+			(xy 71.12 162.56) (xy 73.66 162.56)
 		)
 		(stroke
@@
 	(wire
 		(pts
-			(xy 64.77 168.91) (xy 107.95 168.91)
+			(xy 71.12 168.91) (xy 107.95 168.91)
 		)
 		(stroke
@@
 	(wire
 		(pts
-			(xy 64.77 165.1) (xy 64.77 168.91)
+			(xy 71.12 165.1) (xy 71.12 168.91)
 		)
 		(stroke
@@
 			)
 		)
-		(property "Footprint" "Connector_PinHeader_2.54mm:PinHeader_1x04_P2.54mm_Vertical"
+		(property "Footprint" "Connector_PinSocket_2.54mm:PinSocket_1x04_P2.54mm_Vertical"
 			(at 190.5 93.98 0)
 			(effects
@@
 	(symbol
 		(lib_id "Connector:Conn_01x02_Socket")
-		(at 59.69 162.56 0)
-		(mirror y)
-		(unit 1)
-		(exclude_from_sim no)
-		(in_bom yes)
-		(on_board yes)
-		(dnp no)
-		(property "Reference" "J3"
-			(at 60.325 170.18 0)
-			(effects
-				(font
-					(size 1.27 1.27)
-				)
-			)
-		)
-		(property "Value" "Conn_01x02_Socket"
-			(at 48.514 163.322 0)
-			(effects
-				(font
-					(size 1.27 1.27)
-				)
-				(hide yes)
-			)
-		)
-		(property "Footprint" "TerminalBlock_Phoenix:TerminalBlock_Phoenix_MKDS-1,5-2-5.08_1x02_P5.08mm_Horizontal"
-			(at 59.69 162.56 0)
-			(effects
-				(font
-					(size 1.27 1.27)
-				)
-				(hide yes)
-			)
-		)
-		(property "Datasheet" "~"
-			(at 59.69 162.56 0)
-			(effects
-				(font
-					(size 1.27 1.27)
-				)
-				(hide yes)
-			)
-		)
-		(property "Description" "Generic connector, single row, 01x02, script generated"
-			(at 59.69 162.56 0)
-			(effects
-				(font
-					(size 1.27 1.27)
-				)
-				(hide yes)
-			)
-		)
-		(property "Funktion" "ext. Power 5V DC"
-			(at 50.546 163.83 0)
-			(effects
-				(font
-					(size 1.27 1.27)
-				)
-			)
-		)
-		(pin "1"
-		)
-		(pin "2"
-		)
-		(instances
-			(project "esp32-e22"
-				(path "/7ac59502-473d-4014-a9ef-f4cf3cefb926"
-					(reference "J3")
-					(unit 1)
-				)
-			)
-		)
-	)
-	(symbol
-		(lib_id "Connector:Conn_01x02_Socket")
 		(at 20.32 38.1 0)
 		(mirror y)
@@
 					(unit 1)
 				)
+			)
+		)
+	)
+	(symbol
+		(lib_id "Connector:Screw_Terminal_01x02")
+		(at 66.04 162.56 0)
+		(mirror y)
+		(unit 1)
+		(exclude_from_sim no)
+		(in_bom yes)
+		(on_board yes)
+		(dnp no)
+		(property "Reference" "J3"
+			(at 66.04 168.402 0)
+			(effects
+				(font
+					(size 1.27 1.27)
+				)
+			)
+		)
+		(property "Value" "Screw_Terminal_01x02"
+			(at 63.5 165.0999 0)
+			(effects
+				(font
+					(size 1.27 1.27)
+				)
+				(justify left)
+				(hide yes)
+			)
+		)
+		(property "Footprint" "TerminalBlock_Phoenix:TerminalBlock_Phoenix_MKDS-1,5-2-5.08_1x02_P5.08mm_Horizontal"
+			(at 66.04 162.56 0)
+			(effects
+				(font
+					(size 1.27 1.27)
+				)
+				(hide yes)
+			)
+		)
+		(property "Datasheet" "~"
+			(at 66.04 162.56 0)
+			(effects
+				(font
+					(size 1.27 1.27)
+				)
+				(hide yes)
+			)
+		)
+		(property "Description" "Generic screw terminal, single row, 01x02, script generated (kicad-library-utils/schlib/autogen/connector/)"
+			(at 66.04 162.56 0)
+			(effects
+				(font
+					(size 1.27 1.27)
+				)
+				(hide yes)
+			)
+		)
+		(property "Function" "ext. Power 5V DC"
+			(at 52.832 163.83 0)
+			(effects
+				(font
+					(size 1.27 1.27)
+					(thickness 0.254)
+					(bold yes)
+				)
+			)
+		)
+		(pin "1"
+		)
+		(pin "2"
+		)
+		(instances
+			(project ""
+				(path "/7ac59502-473d-4014-a9ef-f4cf3cefb926"
+					(reference "J3")
+					(unit 1)
+				)

Commit message: update
Parts:
- removed J7: Conn_01x04_Socket, Connector_PinSocket_2.54mm:PinSocket_1x04_P2.54mm_Vertical, symbol Connector:Conn_01x04_Socket
- added J7: Conn_01x05_Socket, Connector_PinSocket_2.54mm:PinSocket_1x05_P2.54mm_Vertical, symbol Connector:Conn_01x05_Socket
- F1: value 5A -> 2A
Connections:
- net +3.3V: now also J7.1 (Pin_1), J7.5 (Pin_5)
- net GND: now also J7.2 (Pin_2)
- net SCL: now also J7.3 (Pin_3)
- net SDA: now also J7.4 (Pin_4)
Other:
- moved on the sheet: C8, JP1, JP2, U2

Commit message: SCH & PCB α5
Parts:
- added D5: 1N4004, Diode_THT:D_DO-41_SOD81_P5.08mm_Vertical_KathodeUp, symbol Diode:1N4004
- added U4: Mini_DC-DC_12-24V_adjustable, KiCad:HW-613, symbol HW-613:Mini_DC-DC_12-24V_adjustable
- D1: footprint Diode_THT:D_DO-41_SOD81_P7.62mm_Horizontal -> Diode_THT:D_DO-41_SOD81_P5.08mm_Vertical_KathodeUp
- J3: Function ext. Power 5V DC -> ext. Power DC
Connections:
- net GND: now also J3.1 (Pin_1), D5.2 (A), U4.2 (GND); no longer J3.2 (Pin_2)
- net at D2.2 (A): now also U4.1 (VO+); no longer F1.2
- net at F1.1: now also J3.2 (Pin_2); no longer J3.1 (Pin_1)
- new net: D5.1 (K), F1.2, U4.3 (IN+)
Other:
- moved on the sheet: C3, C4, C5, D2, D3, D4, F1, J3, R3, R4
