File: ESP32-E22_V2.1.1/KiCad/esp32-e22.kicad_sch (KiCad schematic)
At the start: 44 parts, among them J1 Conn_01x02_Socket, J10 Conn_01x02_Socket, J3 Screw_Terminal_01x02, J4 Conn_01x04_Socket, J5 Conn_01x03_Socket, J6 Conn_01x04_Socket, J7 Conn_01x05_Socket, J8 SMA, J9 Conn_01x02_Socket, SW1 SW_Push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

Commit message: update
Parts:
- U4: value Mini_DC-DC_12-24V_adjustable -> HW-613
Other:
- moved on the sheet: C8, D2, D5, F1, J3, U4

Commit message: update SCH
Parts:
- D5: value 1N4004 -> 1N4007
- J3: Function ext. Power DC -> ext. 6..24V
Other:
- note added: "+"
- note added: "-"
- moved on the sheet: J10
Changed lines of the file:
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@@
 	(title_block
 		(title "ESP32 - E22 Board")
-		(date "2024-10-25")
+		(date "2024-11-03")
 		(rev "V2.1.1")
 		(company "DK9BT / OE3WAS")
@@
 	(wire
 		(pts
-			(xy 49.53 66.04) (xy 49.53 71.12)
+			(xy 49.53 66.04) (xy 49.53 69.85)
 		)
 		(stroke
@@
 	(wire
 		(pts
-			(xy 49.53 73.66) (xy 49.53 77.47)
+			(xy 49.53 72.39) (xy 49.53 77.47)
 		)
 		(stroke
@@
 		)
 	)
+	(text "-"
+		(exclude_from_sim no)
+		(at 49.53 167.894 0)
+		(effects
+			(font
+				(size 1.27 1.27)
+				(thickness 0.254)
+				(bold yes)
+			)
+		)
+	)
 	(text "GPS_TX"
 		(exclude_from_sim no)
@@
 		)
 	)
+	(text "+"
+		(exclude_from_sim no)
+		(at 49.53 164.592 0)
+		(effects
+			(font
+				(size 1.27 1.27)
+				(thickness 0.254)
+				(bold yes)
+			)
+		)
+	)
 	(text "GPS_RX"
 		(exclude_from_sim no)
@@
 	)
 	(label "E22_RXEN"
-		(at 62.23 113.03 0)
+		(at 63.5 113.03 0)
 		(fields_autoplaced yes)
 		(effects
@@
 		(on_board yes)
 		(dnp no)
-		(fields_autoplaced yes)
 		(property "Reference" "#PWR020"
 			(at 270.51 67.31 0)
@@
 		)
 		(property "Value" "GND"
-			(at 273.05 62.2299 0)
+			(at 268.478 65.024 0)
 			(effects
 				(font
@@
 		)
 		(property "Value" "GND"
-			(at 259.08 85.852 0)
+			(at 261.112 86.614 0)
 			(effects
 				(font
@@
 		(on_board yes)
 		(dnp no)
-		(fields_autoplaced yes)
 		(property "Reference" "J1"
-			(at 20.955 35.56 0)
+			(at 20.828 43.18 0)
 			(effects
 				(font
@@
 		(dnp no)
 		(property "Reference" "J3"
-			(at 52.07 161.798 0)
+			(at 51.816 170.942 0)
 			(effects
 				(font
@@
 			)
 		)
-		(property "Function" "ext. Power DC"
+		(property "Function" "ext. 6..24V"
 			(at 43.18 166.37 0)
 			(effects
@@
 	(symbol
 		(lib_id "Connector:Conn_01x02_Socket")
-		(at 44.45 71.12 0)
+		(at 44.45 69.85 0)
 		(mirror y)
 		(unit 1)
@@
 		(on_board yes)
 		(dnp no)
-		(fields_autoplaced yes)
 		(property "Reference" "J10"
-			(at 45.085 68.58 0)
+			(at 45.212 74.422 0)
 			(effects
 				(font
@@
 		)
 		(property "Value" "Conn_01x02_Socket"
-			(at 43.18 73.6599 0)
+			(at 43.18 72.3899 0)
 			(effects
 				(font
@@
 		)
 		(property "Footprint" "Connector_PinHeader_2.54mm:PinHeader_1x02_P2.54mm_Vertical"
-			(at 44.45 71.12 0)
+			(at 44.45 69.85 0)
 			(effects
 				(font
@@
 		)
 		(property "Datasheet" "~"
-			(at 44.45 71.12 0)
+			(at 44.45 69.85 0)
 			(effects
 				(font
@@
 		)
 		(property "Description" "Generic connector, single row, 01x02, script generated"
-			(at 44.45 71.12 0)
+			(at 44.45 69.85 0)
 			(effects
 				(font
@@
 			)
 		)
-		(property "Value" "1N4004"
+		(property "Value" "1N4007"
 			(at 68.58 176.5299 90)
 			(effects
@@
 		(on_board yes)
 		(dnp no)
-		(fields_autoplaced yes)
 		(property "Reference" "J9"
-			(at 278.13 57.1499 0)
+			(at 274.828 60.96 0)
 			(effects
 				(font
