File: ESP32-E22_V2.1.2/KiCad/esp32-e22.kicad_sch (KiCad schematic)
At the start: 45 parts, among them J1 Conn_01x02_Socket, J10 Conn_01x02_Socket, J11 Conn_01x04_Socket, J3 Screw_Terminal_01x02, J4 Conn_01x04_Socket, J5 Conn_01x03_Socket, J6 Conn_01x04_Socket, J7 Conn_01x05_Socket, J8 SMA, J9 Conn_01x02_Socket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

Commit message: update Assembly
Parts:
- J8: footprint Connector_Coaxial:SMA_Amphenol_132134-14_Vertical -> Connector_Coaxial:SMA_Amphenol_901-143_Horizontal
Changed lines of the file:
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@@
 	(title_block
 		(title "ESP32 - E22 Board")
-		(date "2024-11-04")
+		(date "2024-11-05")
 		(rev "V2.1.2")
 		(company "OE3WAS")
@@
 			)
 		)
-		(property "Footprint" "Connector_Coaxial:SMA_Amphenol_132134-14_Vertical"
+		(property "Footprint" "Connector_Coaxial:SMA_Amphenol_901-143_Horizontal"
 			(at 214.63 78.74 0)
 			(effects

Commit message: PCB β3
Parts:
- added J12: Conn_01x02_Socket, Connector_PinHeader_2.54mm:PinHeader_1x02_P2.54mm_Horizontal, symbol Connector:Conn_01x02_Socket
- D5: footprint Diode_THT:D_DO-41_SOD81_P5.08mm_Vertical_KathodeUp -> Diode_THT:D_DO-41_SOD81_P2.54mm_Vertical_KathodeUp
- U1: value ESP32-DevKitC -> ESP32-DevKitC V4
- U3: value E22-40033S -> E22-400M33S
Connections:
- net GND: now also J12.2 (Pin_2)
- net at U4.4 (EN): now also J12.1 (Pin_1)
Other:
- moved on the sheet: D2
Changed lines of the file:
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@@
 	(title_block
 		(title "ESP32 - E22 Board")
-		(date "2024-11-05")
+		(date "2024-11-17")
 		(rev "V2.1.2")
 		(company "OE3WAS")
@@
 	)
 	(junction
+		(at 80.01 186.69)
+		(diameter 0)
+		(color 0 0 0 0)
+	)
+	(junction
 		(at 31.75 186.69)
 		(diameter 0)
@@
 	)
 	(junction
-		(at 100.33 161.29)
-		(diameter 0)
-		(color 0 0 0 0)
-	)
-	(junction
 		(at 149.86 134.62)
 		(diameter 0)
@@
 	)
 	(junction
+		(at 96.52 161.29)
+		(diameter 0)
+		(color 0 0 0 0)
+	)
+	(junction
 		(at 180.34 83.82)
 		(diameter 0)
@@
 	)
 	(junction
+		(at 109.22 161.29)
+		(diameter 0)
+		(color 0 0 0 0)
+	)
+	(junction
 		(at 182.88 88.9)
 		(diameter 0)
@@
 	(wire
 		(pts
-			(xy 46.99 161.29) (xy 100.33 161.29)
+			(xy 46.99 161.29) (xy 96.52 161.29)
 		)
 		(stroke
@@
 	(wire
 		(pts
-			(xy 77.47 186.69) (xy 100.33 186.69)
+			(xy 77.47 186.69) (xy 80.01 186.69)
 		)
 		(stroke
@@
 	(wire
 		(pts
-			(xy 87.63 170.18) (xy 91.44 170.18)
+			(xy 87.63 170.18) (xy 90.17 170.18)
 		)
 		(stroke
@@
 	(wire
 		(pts
+			(xy 80.01 179.07) (xy 80.01 180.34)
+		)
+		(stroke
+			(width 0)
+			(type default)
+		)
+	)
+	(wire
+		(pts
 			(xy 180.34 99.06) (xy 185.42 99.06)
 		)
@@
 	(wire
 		(pts
+			(xy 109.22 161.29) (xy 119.38 161.29)
+		)
+		(stroke
+			(width 0)
+			(type default)
+		)
+	)
+	(wire
+		(pts
 			(xy 95.25 99.06) (xy 95.25 100.33)
 		)
@@
 	(wire
 		(pts
-			(xy 100.33 156.21) (xy 100.33 161.29)
+			(xy 96.52 161.29) (xy 109.22 161.29)
 		)
 		(stroke
@@
 	(wire
 		(pts
-			(xy 100.33 161.29) (xy 100.33 170.18)
+			(xy 80.01 180.34) (xy 83.82 180.34)
+		)
+		(stroke
+			(width 0)
+			(type default)
+		)
+	)
+	(wire
+		(pts
+			(xy 109.22 156.21) (xy 109.22 161.29)
+		)
+		(stroke
+			(width 0)
+			(type default)
+		)
+	)
+	(wire
+		(pts
+			(xy 96.52 161.29) (xy 96.52 170.18)
 		)
 		(stroke
@@
 	(wire
 		(pts
+			(xy 80.01 182.88) (xy 83.82 182.88)
+		)
+		(stroke
+			(width 0)
+			(type default)
+		)
+	)
+	(wire
+		(pts
 			(xy 160.02 161.29) (xy 160.02 165.1)
 		)
@@
 	(wire
 		(pts
+			(xy 80.01 186.69) (xy 100.33 186.69)
+		)
+		(stroke
+			(width 0)
+			(type default)
+		)
+	)
+	(wire
+		(pts
 			(xy 149.86 31.75) (xy 154.94 31.75)
 		)
@@
 	(wire
 		(pts
-			(xy 100.33 161.29) (xy 119.38 161.29)
-		)
-		(stroke
-			(width 0)
-			(type default)
-		)
-	)
-	(wire
-		(pts
 			(xy 177.8 101.6) (xy 185.42 101.6)
 		)
@@
 	(wire
 		(pts
+			(xy 80.01 182.88) (xy 80.01 186.69)
+		)
+		(stroke
+			(width 0)
+			(type default)
+		)
+	)
+	(wire
+		(pts
 			(xy 187.96 53.34) (xy 187.96 58.42)
 		)
@@
 	(wire
 		(pts
-			(xy 96.52 170.18) (xy 100.33 170.18)
+			(xy 95.25 170.18) (xy 96.52 170.18)
 		)
 		(stroke
@@
 	(symbol
 		(lib_id "Device:D_Schottky_Small")
-		(at 93.98 170.18 180)
+		(at 92.71 170.18 180)
 		(unit 1)
 		(exclude_from_sim no)
@@
 		(dnp no)
 		(property "Reference" "D2"
-			(at 94.234 172.72 0)
+			(at 92.964 172.72 0)
 			(effects
 				(font
@@
 		)
 		(property "Value" "1N5817"
-			(at 94.488 174.752 0)
+			(at 93.218 174.752 0)
 			(effects
 				(font
@@
 		)
 		(property "Footprint" "Diode_THT:D_DO-41_SOD81_P7.62mm_Horizontal"
-			(at 93.98 170.18 90)
+			(at 92.71 170.18 90)
 			(effects
 				(font
@@
 		)
 		(property "Datasheet" "~"
-			(at 93.98 170.18 90)
+			(at 92.71 170.18 90)
 			(effects
 				(font
@@
 		)
 		(property "Description" "Schottky diode, small symbol"
-			(at 93.98 170.18 0)
+			(at 92.71 170.18 0)
 			(effects
 				(font
@@
 			)
 		)
-		(property "Value" "ESP32-DevKitC"
-			(at 102.87 99.06 0)
+		(property "Value" "ESP32-DevKitC V4"
+			(at 97.536 103.378 0)
 			(effects
 				(font
-					(size 1.27 1.27)
+					(size 2.54 2.54)
+					(thickness 0.508)
+					(bold yes)
 				)
 				(justify left)
@@
 	(symbol
 		(lib_id "power:+5V")
-		(at 100.33 156.21 0)
+		(at 109.22 156.21 0)
 		(unit 1)
 		(exclude_from_sim no)
@@
 		(dnp no)
 		(property "Reference" "#PWR04"
-			(at 100.33 160.02 0)
+			(at 109.22 160.02 0)
 			(effects
 				(font
@@
 		)
 		(property "Value" "+5V"
-			(at 100.33 151.13 0)
+			(at 109.22 151.13 0)
 			(effects
 				(font
@@
 		)
 		(property "Footprint" ""
-			(at 100.33 156.21 0)
+			(at 109.22 156.21 0)
 			(effects
 				(font
@@
 		)
 		(property "Datasheet" ""
-			(at 100.33 156.21 0)
+			(at 109.22 156.21 0)
 			(effects
 				(font
@@
 		)
 		(property "Description" "Power symbol creates a global label with name \"+5V\""
-			(at 100.33 156.21 0)
+			(at 109.22 156.21 0)
 			(effects
 				(font
@@
 	)
 	(symbol
+		(lib_id "Connector:Conn_01x02_Socket")
+		(at 88.9 180.34 0)
+		(unit 1)
+		(exclude_from_sim no)
+		(in_bom yes)
+		(on_board yes)
+		(dnp no)
+		(property "Reference" "J12"
+			(at 88.138 184.912 0)
+			(effects
+				(font
+					(size 1.27 1.27)
+				)
+			)
+		)
+		(property "Value" "Conn_01x02_Socket"
+			(at 90.17 182.8799 0)
+			(effects
+				(font
+					(size 1.27 1.27)
+				)
+				(justify left)
+				(hide yes)
+			)
+		)
+		(property "Footprint" "Connector_PinHeader_2.54mm:PinHeader_1x02_P2.54mm_Horizontal"
+			(at 88.9 180.34 0)
+			(effects
+				(font
+					(size 1.27 1.27)
+				)
+				(hide yes)
+			)
+		)
+		(property "Datasheet" "~"
+			(at 88.9 180.34 0)
+			(effects
+				(font
+					(size 1.27 1.27)
+				)
+				(hide yes)
+			)
+		)
+		(property "Description" "Generic connector, single row, 01x02, script generated"
+			(at 88.9 180.34 0)
+			(effects
+				(font
+					(size 1.27 1.27)
+				)
+				(hide yes)
+			)
+		)
+		(property "Function" "ext. Pwr.Off"
+			(at 95.504 181.356 0)
+			(effects
+				(font
+					(size 1.27 1.27)
+					(thickness 0.254)
+					(bold yes)
+				)
+			)
+		)
+		(pin "1"
+		)
+		(pin "2"
+		)
+		(instances
+			(project "esp32-e22"
+				(path "/7ac59502-473d-4014-a9ef-f4cf3cefb926"
+					(reference "J12")
+					(unit 1)
+				)
+			)
+		)
+	)
+	(symbol
 		(lib_id "Connector:Screw_Terminal_01x02")
 		(at 52.07 172.72 180)
@@
 		(dnp no)
 		(property "Reference" "U3"
-			(at 245.11 40.005 0)
+			(at 244.856 42.672 0)
 			(effects
 				(font
@@
 			)
 		)
-		(property "Value" "E22-40033S"
-			(at 244.856 42.926 0)
+		(property "Value" "E22-400M33S"
+			(at 241.808 39.116 0)
 			(effects
 				(font
-					(size 1.27 1.27)
+					(size 2.54 2.54)
+					(thickness 0.508)
+					(bold yes)
 				)
 			)
@@
 			)
 		)
-		(property "Footprint" "Diode_THT:D_DO-41_SOD81_P5.08mm_Vertical_KathodeUp"
+		(property "Footprint" "Diode_THT:D_DO-41_SOD81_P2.54mm_Vertical_KathodeUp"
 			(at 61.595 180.34 0)
 			(effects
